File: PowerSupply/TIDA-00746-SchDoc.sch (KiCad schematic (older format))
At the start: 74 parts, among them J18 INPUT, J19 GROUND, Q1 SQJ422EP-T1-GE3, Q2 SQ2360EES-T1-GE3, Q3 SQJ461EP, U11 LM536355QRNL, U12 TLVH431AQDBVRA, U13 LM74610, U14 TPS57114CQRTERQ1, U15 TPS62293TDRVRQ1

Commit message: -Symbole angepasst -Audio Mixing umgezeichnet -Audio Mixing teilweise geprüft
Parts:
- L2, L4: symbol SamacSys_Parts:IHLP3232DZER2R2M11 -> ReleaseDeviceDigitalAudio-rescue:IHLP3232DZER2R2M11-SamacSys_Parts
- L3: symbol SamacSys_Parts:XFL4020-102MEB -> ReleaseDeviceDigitalAudio-rescue:XFL4020-102MEB-SamacSys_Parts
Changed lines of the file:
@@
 $Descr A2 23386 16535
 encoding utf-8
-Sheet 2 2
+Sheet 2 3
 Title "TIDA-00746-SchDoc"
 Date "05 06 2020"
@@
 	21100 12400 21100 12500
 $Comp
-L SamacSys_Parts:IHLP3232DZER2R2M11 L2
+L ReleaseDeviceDigitalAudio-rescue:IHLP3232DZER2R2M11-SamacSys_Parts L2
 U 1 1 60856EC1
 P 8500 10650
@@
 	9300 10650 9900 10650
 $Comp
-L SamacSys_Parts:XFL4020-102MEB L3
+L ReleaseDeviceDigitalAudio-rescue:XFL4020-102MEB-SamacSys_Parts L3
 U 1 1 6085CCC2
 P 17300 6100
@@
 	18100 6100 18350 6100
 $Comp
-L SamacSys_Parts:IHLP3232DZER2R2M11 L4
+L ReleaseDeviceDigitalAudio-rescue:IHLP3232DZER2R2M11-SamacSys_Parts L4
 U 1 1 60888F5C
 P 20100 12200
