File: PowerSupply.sch (KiCad schematic (older format))
At the start: 71 parts

Commit message: - Alles aus rescue Lib noch in neue Lib gepackt
Parts:
- removed Cvcc?: 4.7µF, Capacitor_SMD:C_0805_2012Metric, symbol ReleaseDeviceDigitalAudio-rescue:GCM21BR71C475KA73L--ReleaseDevice-rescue
- added C?: 4u7/16V/X7R, Capacitor_SMD:C_0805_2012Metric, symbol Device:C
Changed lines of the file:
@@
-	1    0    0    -1
-$EndComp
-$Comp
-L ReleaseDeviceDigitalAudio-rescue:GCM21BR71C475KA73L--ReleaseDevice-rescue Cvcc?
-U 1 1 5EDA44AA
-P 4900 13050
-F 0 "Cvcc?" H 4800 13250 60  0000 L BNN
-F 1 "4.7µF" H 4950 13200 50  0000 C CNN
-F 2 "Capacitor_SMD:C_0805_2012Metric" H 4900 13050 50  0001 C CNN
-F 3 "" H 4900 13050 50  0001 C CNN
-F 4 "4.7µF" V -900 12700 60  0001 C CNN "ValueDisplayed"
-	1    4900 13050
 	1    0    0    -1
 $EndComp
@@
 	1    0    0    -1
 $EndComp
+$Comp
+L Device:C C?
+U 1 1 60E76C83
+P 4950 13050
+F 0 "C?" H 5065 13096 50  0000 L CNN
+F 1 "4u7/16V/X7R" H 5065 13005 50  0000 L CNN
+F 2 "Capacitor_SMD:C_0805_2012Metric" H 4988 12900 50  0001 C CNN
+F 3 "~" H 4950 13050 50  0001 C CNN
+	1    4950 13050
+	0    -1   -1   0
+$EndComp
 $EndSCHEMATC

Commit message: PowerSupply update
Parts:
- removed C?: 22pF, Capacitor_SMD:C_0603_1608Metric, symbol Device:C
- removed C?: 10u/10V/X7R, Capacitor_SMD:C_0805_2012Metric, symbol Device:C
- removed R?: 100k/5%, Resistor_SMD:R_0603_1608Metric, symbol Device:R
- removed R?: 100k/1%, Resistor_SMD:R_0603_1608Metric, symbol Device:R
- removed R?: 3R ????????????, Resistor_SMD:R_0603_1608Metric, symbol Device:R
- added C?: 47u/6V3/X5R, Capacitor_SMD:C_1210_3225Metric, symbol Device:C
- added J?: BAT, Connector_PinHeader_2.54mm:PinHeader_1x02_P2.54mm_Horizontal, symbol Connector_Generic:Conn_01x02
- added Q?: SQD50P06-15L_GE3, Package_TO_SOT_SMD:TO-252-2, symbol Device:Q_PMOS_GDS
- L?: footprint footprints:ACM1211 -> TeKaDe:ACM1211
- L? (x2): footprint SamacSys_Parts:INDPM8682X300N -> TeKaDe:IHLP-3232DZ; symbol TeKaDe:IHLP3232DZER2R2M11-SamacSys_Parts -> TeKaDe:IHLP3232DZER2R2M11
- L?: footprint SamacSys_Parts:XFL4020102MEB -> TeKaDe:XLF4020; symbol TeKaDe:XFL4020-102MEB-SamacSys_Parts -> TeKaDe:XFL4020-102MEB
- LF?: footprint footprints:IHLP-2020CZ-11 -> TeKaDe:IHLP-2020CZ-11
- Q?: value SQ2360EES-T1-GE3 -> SQ2362ES-T1_GE3; symbol TeKaDe:SQ2360EES-T1-GE3- -> TeKaDe:SQ2362ES-T1_GE3
- Q?: value SQJ422EP-T1-GE3 -> NVMFS5C442NL; footprint Package_SO:PowerPAK_SO-8_Single -> TeKaDe:ONSemi_SO-8FL_488AA
- Q?: value SQJ461EP -> SQJ461EP-T1-GE3; footprint Package_SO:PowerPAK_SO-8_Single -> TeKaDe:PowerPAK-SO-8L-SINGLE; symbol TeKaDe:SQJ461EP- -> TeKaDe:SQJ461EP-T1-GE3
- R? (x2): value 100k/0.1% -> 100k/1%
- R?: value 249k/0,1% -> 249k/1%
- U?: value TLVH431AQDBVRA -> TLVH431AQDBVRQ1; footprint Package_TO_SOT_SMD:SOT-23-5_HandSoldering -> Package_TO_SOT_SMD:SOT-23-5; symbol TeKaDe:TLVH431AQDBVR_1- -> TeKaDe:TLVH431AQDBVRQ1
- U?: value LM74610 -> LM74610-Q1; symbol TeKaDe:LM74610- -> TeKaDe:LM74610-Q1
- U?: footprint Package_DFN_QFN:WQFN-16-1EP_3x3mm_P0.5mm_EP1.6x1.6mm_ThermalVias -> TeKaDe:TI-PWQFN-N16-1EP
- U?: value LM536355QRNL -> LM53635LQRNL*Q1; footprint footprints:LM536253QRNLRQ1 -> TeKaDe:TI-VQFN-HR
- U?: footprint DRV6_1P6X1 -> TeKaDe:TI-WSON-6-1EP
Connections:
- net labels added: VSNS
- net labels removed: VSNS1
- wire segments 288 -> 285
- no-connect marks 0 -> 1
Other:
- note added: "1.8V / 1A fixed out\nFPWM aktiv -> f_sw immer 2,25 MHz\n\nAusgangsspannung Ripple: 0,31mV\nStormbedarf am Ausgang: 400mA\n(lt 20210617 Leistungsaufnahme.xlsx)\n\nSpule etwas überdimensioniert, 2u2 / 40mR / 2.6A würde reichen\n\n\nÄnderungen:\n22p C entfernt, nur bei adjustable Typen notwendig\n(Überprüft mit Webbench und DS vgl. S.3 / FB Pin Beschreibung)\nMode auf High -> FPWM Mode\nCout von 10u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"
- note added: "1u / 11mR / 5A"
- note added: "2u2 / 9mR / 10A"
- note added: "3.3V / 3A\nR an RT/CLK = 82k5 -> f_sw 2,0 MHz\nC an SS/TR = 10n -> Slowstart Rate 4ms (Cout muss geladen werden)\n\nAusgangsspannung Ripple: 0,21mV\nStormbedarf am Ausgang: 800mA\n(lt 20210617 Leistungsaufnahme.xlsx)\n\nÄnderungen:\nFeedback R Toleranz auf 1% (war unnötigerweise 0,1)\nGND und GNDA getrennt"
- note added: "5V / 3,5A fixed out\nFPWM aktiv -> f_sw immer 2,1 MHz\n\nAusgangsspannung Ripple: 0,45mV\nStormbedarf am Ausgang: 2600mA\n(lt 20210617 Leistungsaufnahme.xlsx)\n\nÄnderungen:\nRbias entfernt, nur notwendig wenn langes Kabel am Ausgang. Vgl. DS 9.2.1.2.4\nReset Pullup entfernt, Reset Ausgang wird nicht verwendet, floating. Vgl. DS 8.3.1\nFPWM Input via VCC auf High ziehen, vgl. DS 9.2.1.2.3\nEN ohn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"
- note added: "COMP Beschaltung wie in Evalboard\nWebbench Designer liefert folgende Werte:\n(5k76 + 2n2) | 110p"
- note added: "LM74510 Layout\n"
- note added: "Max. 36VDC\n"
- note added: "Max. 6VDC\n"
- note added: "Place bypass capacitors for VCC and BIAS close\nto their respective pins. \n\nMake sure AGND pin “sees” the CVCC and CBIAS \ncapacitors first before connecting it to GND.\n\nUse dedicated feedback trace and away from \nswitch node and CBOOT capacitor to avoid any\ncross coupling into sensitive analog feedback."
- note added: "Steckverbinder KFZ Spannungseingang"
- note added: "Tie the GND pins and AGND pin directly to the\nthermal pad under the IC. \n\nConnect the thermal pad to any internal PCB ground \nlanes using multiple vias directly under the IC."
- note added: "Änderungen:\nToleranz der 100k Rs auf 1%, war unnötigerweise 0,1%\nSQ2360EES-T1-GE3 durch SQ2362ES-T1_GE3 ersetzt (wie vom Hersteller empfohlen)\nSQJ422EP-T1-GE3 durch NVMFS5C442NL ersetzt (ONSemi_SO-8FL_488AA Footprint)\nSQJ461EP-T1-GE3 durch SQD50P06-15L_GE3 ersetzt (TO-252 Footprint)"
- note removed: "1.8V\n"
- note removed: "3.3V\n"
- note removed: "5V\n"
- note removed: "Achtung Steckverbinder fehlt\n"
- note removed: "Den hier komplett checken"
- note removed: "RESET Beschaltung checken, in Evalboard gehts hier auf Brücke"
- note removed: "Warum 100k Rs an den SQs 0.1%??\n"
- note removed: "fsw=2Mhz"
- moved on the sheet: C?, D?, L?, LF?, Q?, R?, U?
