File: RaspberryPiCM.sch (KiCad schematic (older format))
At the start: 13 parts

Commit message: Mehr Hierarchie
Parts:
- added BT?: Battery, Connectors:CR1220, symbol Device:Battery
- added C?: 1uF, Capacitor_SMD:C_0603_1608Metric, symbol Device:C
- added U?: DS3231M, Package_SO:SOIC-16W_7.5x10.3mm_P1.27mm, symbol Timer_RTC:DS3231M
Connections:
- net +3V3: now also C?.1, U?.2 (VCC)
- net Earth: now also BT?.2 (-), C?.2, U?.10 (GND), U?.11 (GND), U?.12 (GND), U?.13 (GND), U?.5 (GND), U?.6 (GND), U?.7 (GND), U?.8 (GND), U?.9 (GND)
- net Rpi.SCL1: now also U?.16 (SCL)
- net Rpi.SDA1: now also U?.15 (SDA)
- new net: BT?.1 (+), U?.14 (VBAT)
- no-connect marks 2 -> 5
Other:
- note added: "Clock"
Changed lines of the file:
@@
 $Descr A2 23386 16535
 encoding utf-8
-Sheet 4 5
+Sheet 2 7
 Title ""
 Date ""
@@
 NoConn ~ 5700 750
 NoConn ~ 5700 7500
-Text Label 1850 1350 2    50   ~ 0
+Text Label 1450 1350 2    50   ~ 0
 Rpi.SDA1
-Text Label 1850 1500 2    50   ~ 0
+Text Label 1450 1500 2    50   ~ 0
 Rpi.SCL1
 Text Label 1050 6150 0    50   ~ 0
@@
 Wire Wire Line
 	1150 3150 3700 3150
-Text HLabel 1150 1250 0    50   BiDi ~ 0
-I2C1
-Entry Wire Line
-	1350 1250 1450 1350
 Wire Wire Line
 	1450 1350 3700 1350
-Entry Wire Line
-	1350 1400 1450 1500
 Wire Wire Line
 	1450 1500 3700 1500
-Wire Bus Line
-	1150 1250 1350 1250
-Wire Bus Line
-	1350 1250 1350 1400
 Text Label 1550 4800 2    50   ~ 0
 RPi_UART_RX
@@
 	1    0    0    -1
 $EndComp
+$Comp
+L Timer_RTC:DS3231M U?
+U 1 1 60ED0E56
+P 18900 3050
+AR Path="/60ED0E56" Ref="U?"  Part="1"
+AR Path="/614D7E9D/60ED0E56" Ref="U?"  Part="1"
+F 0 "U?" H 18900 2561 50  0000 C CNN
+F 1 "DS3231M" H 18900 2470 50  0000 C CNN
+F 2 "Package_SO:SOIC-16W_7.5x10.3mm_P1.27mm" H 18900 2450 50  0001 C CNN
+F 3 "http://datasheets.maximintegrated.com/en/ds/DS3231.pdf" H 19170 3100 50  0001 C CNN
+F 4 "good" H 18900 3050 50  0001 C CNN "Availability"
+	1    18900 3050
+	1    0    0    -1
+$EndComp
+$Comp
+L Device:Battery BT?
+U 1 1 60ED0E5C
+P 19900 2950
+AR Path="/60ED0E5C" Ref="BT?"  Part="1"
+AR Path="/614D7E9D/60ED0E5C" Ref="BT?"  Part="1"
+F 0 "BT?" H 20008 2996 50  0000 L CNN
+F 1 "Battery" H 20008 2905 50  0000 L CNN
+F 2 "Connectors:CR1220" V 19900 3010 50  0001 C CNN
+F 3 "~" V 19900 3010 50  0001 C CNN
+	1    19900 2950
+	1    0    0    -1
+$EndComp
+Wire Wire Line
+	18900 2650 18900 2550
+Wire Wire Line
+	18900 2550 19900 2550
+Wire Wire Line
+	19900 2550 19900 2750
+Wire Wire Line
+	19900 3150 19900 3550
+Wire Wire Line
+	19900 3550 18900 3550
+Wire Wire Line
+	18900 3550 18900 3450
+NoConn ~ 19400 2850
+NoConn ~ 19400 3150
+NoConn ~ 18400 3250
+$Comp
+L power:+3.3V #PWR?
+U 1 1 60ED0E6B
+P 18800 2350
+F 0 "#PWR?" H 18800 2200 50  0001 C CNN
+F 1 "+3.3V" H 18815 2523 50  0000 C CNN
+F 2 "" H 18800 2350 50  0001 C CNN
+F 3 "" H 18800 2350 50  0001 C CNN
+	1    18800 2350
+	1    0    0    -1
+$EndComp
+Wire Wire Line
+	18800 2350 18800 2450
+$Comp
+L Device:C C?
+U 1 1 60ED0E72
+P 18550 2450
+F 0 "C?" V 18298 2450 50  0000 C CNN
+F 1 "1uF" V 18389 2450 50  0000 C CNN
+F 2 "Capacitor_SMD:C_0603_1608Metric" H 18588 2300 50  0001 C CNN
+F 3 "~" H 18550 2450 50  0001 C CNN
+	1    18550 2450
+	0    1    1    0
+$EndComp
+$Comp
+L power:Earth #PWR?
+U 1 1 60ED0E78
+P 18100 2500
+F 0 "#PWR?" H 18100 2250 50  0001 C CNN
+F 1 "Earth" H 18100 2350 50  0001 C CNN
+F 2 "" H 18100 2500 50  0001 C CNN
+F 3 "~" H 18100 2500 50  0001 C CNN
+	1    18100 2500
+	1    0    0    -1
+$EndComp
+$Comp
+L power:Earth #PWR?
+U 1 1 60ED0E7E
+P 19900 3700
+F 0 "#PWR?" H 19900 3450 50  0001 C CNN
+F 1 "Earth" H 19900 3550 50  0001 C CNN
+F 2 "" H 19900 3700 50  0001 C CNN
+F 3 "~" H 19900 3700 50  0001 C CNN
+	1    19900 3700
+	1    0    0    -1
+$EndComp
+Wire Wire Line
+	19900 3700 19900 3550
+Connection ~ 19900 3550
+Wire Wire Line
+	18800 2450 18700 2450
+Connection ~ 18800 2450
+Wire Wire Line
+	18800 2450 18800 2650
+Wire Wire Line
+	18400 2450 18100 2450
+Wire Wire Line
+	18100 2450 18100 2500
+Text Label 17850 2950 2    50   ~ 0
+Rpi.SDA1
+Text Label 17850 2850 2    50   ~ 0
+Rpi.SCL1
+Wire Wire Line
+	18400 2950 17850 2950
+Wire Wire Line
+	17850 2850 18400 2850
+Wire Notes Line
+	20350 1900 20350 4150
+Wire Notes Line
+	20350 4150 17400 4150
+Wire Notes Line
+	17400 4150 17400 1900
+Wire Notes Line
+	17400 1900 20350 1900
+Text Notes 17600 2150 0    50   ~ 0
+Clock
 Wire Bus Line
 	900  5450 900  6050
