File: ReleaseDeviceDigitalAudio.sch (KiCad schematic (older format))
At the start: 5 parts, among them J1 AudioJack3, J2 AudioJack3, J3 AudioJack3, J4 AudioJack3, J5 AudioJack3

Commit message: [fix:] general troublespots -> notes
Changed lines of the file:
@@
 NoConn ~ 3100 -2600
 NoConn ~ 3100 -2500
-Text Notes 5750 8250 1    50   ~ 0
+Text Notes 5650 7850 1    50   ~ 0
 RPi NOT 5V tolerant!
 $Sheet
@@
 F11 "7Seg_Decoder_D1" O R 9650 6850 50
 F12 "BrightnessPWM" O R 9650 6650 50
-F13 "RPI_RUN" O L 8050 6650 50
+F13 "RPI_RUN" O L 8050 8450 50
 F14 "UART1_RX" I L 8050 6950 50
 F15 "UART1_TX" O L 8050 7050 50
@@
 F2 "GPIO9" O R 5550 4900 50
 F3 "GPIO10" I R 5550 1700 50
-F4 "RUN" I R 5550 6650 50
+F4 "RUN" I R 5550 8450 50
 F5 "I2C0_SDA" B R 5550 5700 50
 F6 "I2C1_SDA" B R 5550 1400 50
@@
 I2S Slave
 Wire Wire Line
-	6200 6650 5550 6650
-Wire Wire Line
-	8050 6650 7400 6650
-Wire Wire Line
 	7400 7050 8050 7050
 Wire Wire Line
@@
 F0 "LevelShift" 50
 F1 "LevelShift.sch" 50
-F2 "RUN_3V3" O L 6200 6650 50
-F3 "RUN_5V" I R 7400 6650 50
-F4 "UART_TX_5V" I R 7400 7050 50
-F5 "UART_TX_3V3" O L 6200 7050 50
-F6 "UART_RX_5V" O R 7400 6950 50
-F7 "UART_RX_3V3" I L 6200 6950 50
+F2 "UART_TX_5V" I R 7400 7050 50
+F3 "UART_TX_3V3" O L 6200 7050 50
+F4 "UART_RX_5V" O R 7400 6950 50
+F5 "UART_RX_3V3" I L 6200 6950 50
 $EndSheet
 Wire Wire Line
@@
 $EndComp
 Text Notes 900  5800 0    50   ~ 0
-Allgemeines: \n- Levelshift prüfen (Zuordnung RX/TX)\n- Signalzuordungen I2C / I2S / UART checken\n- Steckverbinder KFZ (Dauerstrom / Zündung)\n- Steckverbinder Analog Audio\n- Footprint Q von Dauerstrom Verpolschutz machen\n\nSelbsthaltung:\n- Verhalten GPIO output bei undervoltage lockout\n- Zündung nur 1pol anschließen? -> kein Verpolschutz notwendig\n  (Optokoppler Eingang verträgt nur 5V reverse...)\n- Test (Simulation wäre zu aufwendig)\n\nBM83:\n- Warum Temperatur messen?\n- Unused Pin Connections nicht beschrieben\n- MFB wird noch getestet durch Fredrik\n\nMAX98089:\n- LDO für MAX98089?\n\nRTC:\n- Battery Holder so ok (CR1220)?\n\nCM4: \n- RUN PG / Global_EN Test durch Fredrik\n- Footprint checken durch Fredrik\n- Checken ob die 3,3 und 1,8V ausgänge bzgl. Ripple in Ordnung sind\n- Schaltfrequenz onboard Regler\n\nATmega:\n- Wozu 10k R an PWM Ausgang?\n   -> 1V macht Vollaussteuerung\n        Fredrik klärt PWM Frequenz, Auflöung und Eingangs-R des Zeigers\n- int. OSC checken bzgl. Kalwerte und UART Baudrate\n    -> macht Fredrik\n- Programmierbeschaltung ohne Reset?\n    -> check durch Fredrik\n- Auslegung Vorwiderstände an reale LEDs\n- Auslegung Spannungsteiler mit LDR\n
+Allgemeines: \n- Levelshift prüfen (Zuordnung RX/TX)\n- Signalzuordungen I2C / I2S / UART checken\n- Steckverbinder KFZ (Dauerstrom / Zündung)\n- Steckverbinder Analog Audio\n- Footprint Q von Dauerstrom Verpolschutz machen\n\nSelbsthaltung:\n- Verhalten GPIO output bei undervoltage lockout\n- Zündung nur 1pol anschließen? -> kein Verpolschutz notwendig\n  (Optokoppler Eingang verträgt nur 5V reverse...)\n- Test (Simulation wäre zu aufwendig)\n\nBM83:\n- Warum Temperatur messen?\n- Unused Pin Connections nicht beschrieben\n- MFB wird noch getestet durch Fredrik\n\nMAX98089:\n- LDO für MAX98089? \n    - Test: Stromversorgung über CM: kein Noise, Load unerheblich\n-Config: Voice vs. Music filter: Done\n\n\nRTC:\n- Battery Holder so ok (CR1220)?\n\nCM4: \n- RUN PG / Global_EN Test durch Fredrik\n    -> 5V-Kompatibel -> LevelShift entfällt\n- Footprint checken durch Fredrik\n    -> Passt perfekt\n- Checken ob die 3,3 und 1,8V ausgänge bzgl. Ripple in Ordnung sind\n    -> Für MAX98089 ausreichend, Oszilloskop fehlt, daher keine genauen Daten\n- Schaltfrequenz onboard Regler\n    -> 1 - 2.1 MHz (abhängig von Config)\n\nATmega:\n- Wozu 10k R an PWM Ausgang?\n   -> 1V macht Vollaussteuerung\n        Fredrik klärt PWM Frequenz, Auflöung und Eingangs-R des Zeigers\n        -> Vollaussteuerung bei 0.22V, 0.5-1k Eigenwiderstand -> 15k Vorwiderstand (geprüft)\n        -> PER=100 -> 0,05V-Schritte, f=100kHz\n- int. OSC checken bzgl. Kalwerte und UART Baudrate\n    -> macht Fredrik\n- Programmierbeschaltung ohne Reset?\n    -> check durch Fredrik\n- Auslegung Vorwiderstände an reale LEDs\n- Auslegung Spannungsteiler mit LDR\n
 Wire Wire Line
 	9650 2400 12850 2400
@@
 Text Notes 11000 8300 0    50   ~ 0
 IO Voltage: 5V
+Wire Wire Line
+	8050 8450 5550 8450
 $EndSCHEMATC

Commit message: - Kommentare aktualisiert
Changed lines of the file:
@@
 $EndComp
 Text Notes 900  5800 0    50   ~ 0
-Allgemeines: \n- Levelshift prüfen (Zuordnung RX/TX)\n- Signalzuordungen I2C / I2S / UART checken\n- Steckverbinder KFZ (Dauerstrom / Zündung)\n- Steckverbinder Analog Audio\n- Footprint Q von Dauerstrom Verpolschutz machen\n\nSelbsthaltung:\n- Verhalten GPIO output bei undervoltage lockout\n- Zündung nur 1pol anschließen? -> kein Verpolschutz notwendig\n  (Optokoppler Eingang verträgt nur 5V reverse...)\n- Test (Simulation wäre zu aufwendig)\n\nBM83:\n- Warum Temperatur messen?\n- Unused Pin Connections nicht beschrieben\n- MFB wird noch getestet durch Fredrik\n\nMAX98089:\n- LDO für MAX98089? \n    - Test: Stromversorgung über CM: kein Noise, Load unerheblich\n-Config: Voice vs. Music filter: Done\n\n\nRTC:\n- Battery Holder so ok (CR1220)?\n\nCM4: \n- RUN PG / Global_EN Test durch Fredrik\n    -> 5V-Kompatibel -> LevelShift entfällt\n- Footprint checken durch Fredrik\n    -> Passt perfekt\n- Checken ob die 3,3 und 1,8V ausgänge bzgl. Ripple in Ordnung sind\n    -> Für MAX98089 ausreichend, Oszilloskop fehlt, daher keine genauen Daten\n- Schaltfrequenz onboard Regler\n    -> 1 - 2.1 MHz (abhängig von Config)\n\nATmega:\n- Wozu 10k R an PWM Ausgang?\n   -> 1V macht Vollaussteuerung\n        Fredrik klärt PWM Frequenz, Auflöung und Eingangs-R des Zeigers\n        -> Vollaussteuerung bei 0.22V, 0.5-1k Eigenwiderstand -> 15k Vorwiderstand (geprüft)\n        -> PER=100 -> 0,05V-Schritte, f=100kHz\n- int. OSC checken bzgl. Kalwerte und UART Baudrate\n    -> macht Fredrik\n- Programmierbeschaltung ohne Reset?\n    -> check durch Fredrik\n- Auslegung Vorwiderstände an reale LEDs\n- Auslegung Spannungsteiler mit LDR\n
+Allgemeines: \n- Levelshift prüfen (Zuordnung RX/TX)\n- Signalzuordungen I2C / I2S / UART checken\n- Steckverbinder KFZ (Dauerstrom / Zündung)\n- Steckverbinder Analog Audio\n- Footprint Q von Dauerstrom Verpolschutz machen\n\nSelbsthaltung:\n- Verhalten GPIO output bei undervoltage lockout\n- Zündung nur 1pol anschließen? -> kein Verpolschutz notwendig\n  (Optokoppler Eingang verträgt nur 5V reverse...)\n- Test (Simulation wäre zu aufwendig)\n\nBM83:\n- Ersetzen durch Modell mit automotive Zulassung?\n- Warum Temperatur messen?\n- Unused Pin Connections nicht beschrieben\n- MFB wird noch getestet durch Fredrik\n- Microchip Design Checklist ausfuellen, wenn Layout fertig\n\nRTC:\n- Battery Holder CR1220 ? Layout wirds zeigen...\n\nATmega:\n- int. OSC checken bzgl. Kalwerte und UART Baudrate\n    -> macht Fredrik\n- Programmierbeschaltung ohne Reset?\n    -> check durch Fredrik\n- Auslegung Vorwiderstände an reale LEDs\n- Auslegung Spannungsteiler mit LDR\n\n\n\n\nERLEDIGT:\nCM4: \n- RUN PG / Global_EN Test durch Fredrik\n    -> 5V-Kompatibel -> LevelShift entfällt (GETESTET)\n- Footprint checken durch Fredrik\n    -> Passt perfekt (GETESTET)\n- Checken ob die 3,3 und 1,8V ausgänge bzgl. Ripple in Ordnung sind\n    -> Für MAX98089 ausreichend, Oszi fehlt, daher keine genauen Daten\n- Schaltfrequenz onboard Regler\n    -> 1 - 2.1 MHz (abhängig von Config)\n\nMAX98089:\n- LDO für MAX98089? \n    - Test: Stromversorgung über CM: kein Noise, Load unerheblich\n- Config: Voice vs. Music filter: Done\n\nATmega:\n- Wozu 10k R an PWM Ausgang?\n   -> 1V macht Vollaussteuerung\n        Fredrik klärt PWM Frequenz, Auflöung und Eingangs-R des Zeigers\n        -> Vollausst. bei 0.22V, 0.5-1k R_innen -> 15k Vorwiderstand (GETESTET)\n        -> PER=100 -> 0,05V-Schritte, f=100kHz\n\n
 Wire Wire Line
 	9650 2400 12850 2400
