File: UIBoardStandalone.sch (KiCad schematic (older format))
At the start: 45 parts, among them J10 Conn_02x15_Odd_Even, J17 Conn_02x08_Odd_Even, SW1 Button_P, SW10 Button_4, SW11 Button_8, SW12 Button_0, SW13 Button_2, SW14 Button_5, SW15 Button_3, SW16 Button_6, SW17 Button_9, SW18 Button_Z, SW2 Button_X, SW3 Button_S, SW4 Button_G, SW5 Button_R, SW6 Button_M, SW7 Button_7, SW8 Button_Y, SW9 Button_1, U10 MM74C923

Commit message: - Kommentare aktualisiert
Other:
- note added: "Footprint 7Seg machen\n\nTaster spezifizieren\nLEDs spezifizieren (3 oder 5mm bedrahtet, Montagehöhe)\nLDR spezifizieren (bedrahtet, Montagehöhe)\nZiffernblock Backlight??\nSignalStrength / Keyswitch connectoren?\n\nÄnderungen:\n- OnSwitchLedAnode durch 5V ersetzt\n- Footprint Konnektoren MALE"
- note removed: "SignalStrength / Keyswitch connectoren?\n\nÄnderungen:\n- OnSwitchLedAnode durch 5V ersetzt\n- Footprint Konnektoren MALE"
- moved on the sheet: C85, C86, C?, D1, D2, D3, D4, J10, J17, R61, SW1, SW10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

Commit message: - Footprint HD1077R
Parts:
- removed U? (x15): HD1077R, symbol TeKaDe:HD1077R
- added U11, U12, U13, U14, U15, U16, U17, U2, U3, U4, U5, U6, U7, U8, U9: HD1077R, TeKaDe:7SegmentLED_HD1077R, symbol TeKaDe:HD1077R
- D1, D2, D3: footprint (none) -> LED_THT:LED_D5.0mm
- D4: footprint (none) -> LED_THT:LED_D3.0mm
- R61: footprint (none) -> OptoDevice:R_LDR_4.9x4.2mm_P2.54mm_Vertical
- U1: renamed from U?; footprint (none) -> TeKaDe:7SegmentLED_HD1077R
- gave numbers to parts that had none: 1
Connections:
- net AnodeSegmentA: now also U11.7 (a), U12.7 (a), U13.7 (a), U14.7 (a), U15.7 (a), U16.7 (a), U17.7 (a), U2.7 (a), U3.7 (a), U4.7 (a), U5.7 (a), U6.7 (a), U7.7 (a), U8.7 (a), U9.7 (a)
- net AnodeSegmentB: now also U11.6 (b), U12.6 (b), U13.6 (b), U14.6 (b), U15.6 (b), U16.6 (b), U17.6 (b), U2.6 (b), U3.6 (b), U4.6 (b), U5.6 (b), U6.6 (b), U7.6 (b), U8.6 (b), U9.6 (b)
- net AnodeSegmentC: now also U11.4 (c), U12.4 (c), U13.4 (c), U14.4 (c), U15.4 (c), U16.4 (c), U17.4 (c), U2.4 (c), U3.4 (c), U4.4 (c), U5.4 (c), U6.4 (c), U7.4 (c), U8.4 (c), U9.4 (c)
- net AnodeSegmentD: now also U11.2 (d), U12.2 (d), U13.2 (d), U14.2 (d), U15.2 (d), U16.2 (d), U17.2 (d), U2.2 (d), U3.2 (d), U4.2 (d), U5.2 (d), U6.2 (d), U7.2 (d), U8.2 (d), U9.2 (d)
- net AnodeSegmentE: now also U11.1 (e), U12.1 (e), U13.1 (e), U14.1 (e), U15.1 (e), U16.1 (e), U17.1 (e), U2.1 (e), U3.1 (e), U4.1 (e), U5.1 (e), U6.1 (e), U7.1 (e), U8.1 (e), U9.1 (e)
- net AnodeSegmentF: now also U11.10 (f), U12.10 (f), U13.10 (f), U14.10 (f), U15.10 (f), U16.10 (f), U17.10 (f), U2.10 (f), U3.10 (f), U4.10 (f), U5.10 (f), U6.10 (f), U7.10 (f), U8.10 (f), U9.10 (f)
- net AnodeSegmentG: now also U11.9 (g), U12.9 (g), U13.9 (g), U14.9 (g), U15.9 (g), U16.9 (g), U17.9 (g), U2.9 (g), U3.9 (g), U4.9 (g), U5.9 (g), U6.9 (g), U7.9 (g), U8.9 (g), U9.9 (g)
- net CathodeDigit10: now also U11.3 (K)
- net CathodeDigit11: now also U12.3 (K)
- net CathodeDigit12: now also U13.3 (K)
- net CathodeDigit13: now also U14.3 (K)
- net CathodeDigit14: now also U15.3 (K)
- net CathodeDigit2: now also U2.3 (K)
- net CathodeDigit3: now also U3.3 (K)
- net CathodeDigit4: now also U4.3 (K)
- net CathodeDigit5: now also U5.3 (K)
- net CathodeDigit6: now also U6.3 (K)
- net CathodeDigit7: now also U7.3 (K)
- net CathodeDigit8: now also U8.3 (K)
- net CathodeDigit9: now also U9.3 (K)
- net CathodeDigitA: now also U16.3 (K)
- net CathodeDigitB: now also U17.3 (K)
Other:
- note added: "Footprint HD1077R prüfen\n\nLED Farbzuordnung prüfen\nTaster spezifizieren\nLEDs spezifizieren (3 oder 5mm bedrahtet, Montagehöhe)\nLDR spezifizieren (bedrahtet, Montagehöhe)\nZiffernblock Backlight??\nSignalStrength / Keyswitch connectoren?\n\nÄnderungen:\n- OnSwitchLedAnode durch 5V ersetzt\n- Footprint Konnektoren MALE\n- Footprint HD1077R"
- note removed: "Footprint 7Seg machen\n\nTaster spezifizieren\nLEDs spezifizieren (3 oder 5mm bedrahtet, Montagehöhe)\nLDR spezifizieren (bedrahtet, Montagehöhe)\nZiffernblock Backlight??\nSignalStrength / Keyswitch connectoren?\n\nÄnderungen:\n- OnSwitchLedAnode durch 5V ersetzt\n- Footprint Konnektoren MALE"
