File: UIBoardStandalone.sch (KiCad schematic (older format))
At the start: 61 parts, among them J1 Conn_02x08_Odd_Even, J2 Conn_02x15_Odd_Even, SW1 Button_X, SW10 Button_6, SW11 Button_S, SW12 Button_7, SW13 Button_8, SW14 Button_9, SW15 Button_G, SW16 Button_Y, SW17 Button_0, SW18 Button_Z, SW2 Button_R, SW3 Button_1, SW4 Button_2, SW5 Button_3, SW6 Button_P, SW7 Button_M, SW8 Button_4, SW9 Button_5, U1 HD1077R, U10 HD1077R, U11 HD1077R, U12 HD1077R, U13 HD1077R, U14 HD1077R, U15 HD1077R, U16 HD1077R, U17 MM74C923, U2 HD1077R, U3 HD1077R, U4 HD1077R, U5 HD1077R, U6 HD1077R, U7 HD1077R, U8 HD1077R, U9 HD1077R

Commit message: - Erster Stand UI Board Layout
Parts:
- removed R? (x4): 1.25k, symbol Device:R
- added R3, R4, R5, R6: tbd, Resistor_SMD:R_0603_1608Metric, symbol Device:R
- C1: value 100n/10V/X7R -> 100n/16V/X5R; footprint Resistor_SMD:R_0603_1608Metric -> Capacitor_SMD:C_0603_1608Metric
- C2: value 2u2 / 10V / X5R -> 2u2/10V/X5R; footprint (none) -> Capacitor_SMD:C_0603_1608Metric
- C3: value 220n / 10V / X5R -> 220n/10V/X5R; footprint (none) -> Capacitor_SMD:C_0603_1608Metric
- R2: renamed from R?; value 1.25k -> tbd; footprint (none) -> Resistor_SMD:R_0603_1608Metric
- SW1, SW10, SW11, SW12, SW13, SW14, SW15, SW16, SW17, SW18, SW2, SW3, SW4, SW5, SW6, SW7, SW8, SW9: footprint Button_Switch_SMD:SW_SPST_EVQP0 -> TeKaDe:SW_Push_CK_KST2x1G
- U17: value MM74C923 -> MM74C923WM; Distributor (none) -> https://www.aeri.com/products/search/?q=mm74c923
Connections:
- net +5V: no longer J2.30 (Pin_30), R2.1
- net at D6.2 (A): now also R3.2
- net at D7.2 (A): now also R4.2
- net at D8.2 (A): now also R5.2
- net at D9.2 (A): now also R6.2
- new net +5VA: J2.30 (Pin_30), R2.1, R3.1, R4.1, R5.1, R6.1
Other:
- note added: "Backlight Schaltbar"
- note added: "KONSTANT\n"
- note added: "TODO FREDRIK:\n- Bauteil "Schloss" definieren mit Abmessungen und el. Anschlüssen -> erledigt\n- Backlight LED spezifizieren, damit Vorwiderstand ausgelegt werden kann\n- LDR spezifizieren\n\nERLEDIGT:\nLED Farbzuordnung prüfen\n -> stimmt\nTaster spezifizieren\n -> 5mm Gesamthöhe, 0,5mm Tastenhub\nLEDs spezifizieren (3 oder 5mm bedrahtet, Montagehöhe)\n -> Montagehöhe jeweils als Field hinzugefü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"
- note removed: "TODO ALEX:\n- Abschaltung UI Board implementieren (SW6 soll 5V von UI Board schalten, LED_ON alternierend dazu\n- Button Footprint machen:\nhttps://www.digikey.de/product-detail/de/KST241JLFS/401-1850-1-ND/1003967?itemSeq=376558534\nhttps://www.digikey.de/product-detail/de/c-k/KST221JLFS/401-1848-1-ND/1003965\nhttps://www.digikey.de/product-detail/de/1571634-2/450-2408-1-ND/6810844?itemSeq=376561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"
- note removed: "https://www.aeri.com/products/search/?q=hd1077\n"
- note removed: "https://www.aeri.com/products/search/?q=mm74c923\n"
- moved on the sheet: D1, D2, D3, D4, D5, D6, D7, D8, D9, J2, R1, R2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

Commit message: [add:] LED specifications
Parts:
- D5, D6, D7, D8, D9: Digikey Part Number (none) -> 1516-QBL7IW60D-WW-ND
Changed lines of the file:
@@
 F 1 "LED_RD" V 10788 4330 50  0000 L CNN
 F 2 "LED_THT:LED_D5.0mm" H 10750 4250 50  0001 C CNN
-F 3 "~" H 10750 4250 50  0001 C CNN
+F 3 "https://www.aopled.com/AOP_PDFs/L513SRD-B.pdf" H 10750 4250 50  0001 C CNN
 F 4 "9mm" V 10750 4250 50  0001 C CNN "Montagehöhe"
 	1    10750 4250
@@
 F 1 "LED_YL" V 10288 4330 50  0000 L CNN
 F 2 "LED_THT:LED_D5.0mm" H 10250 4250 50  0001 C CNN
-F 3 "~" H 10250 4250 50  0001 C CNN
+F 3 "https://media.digikey.com/pdf/Data%20Sheets/Lite-On%20PDFs/LTL-4273.pdf" H 10250 4250 50  0001 C CNN
 F 4 "9mm" V 10250 4250 50  0001 C CNN "Montagehöhe"
 	1    10250 4250
@@
 F 1 "LED_GN" V 9638 4330 50  0000 L CNN
 F 2 "LED_THT:LED_D5.0mm" H 9600 4250 50  0001 C CNN
-F 3 "~" H 9600 4250 50  0001 C CNN
+F 3 "https://www.aopled.com/AOP_PDFs/L513GD-B.pdf" H 9600 4250 50  0001 C CNN
 F 4 "9mm" V 9600 4250 50  0001 C CNN "Montagehöhe"
 	1    9600 4250
@@
 F 1 "LED_ON" V 11288 4330 50  0000 L CNN
 F 2 "LED_THT:LED_D3.0mm" H 11250 4250 50  0001 C CNN
-F 3 "~" H 11250 4250 50  0001 C CNN
+F 3 "https://media.digikey.com/pdf/Data%20Sheets/Lite-On%20PDFs/LTL-1CHYE.pdf" H 11250 4250 50  0001 C CNN
 F 4 "8mm" V 11250 4250 50  0001 C CNN "Montagehöhe"
 	1    11250 4250
@@
 $EndComp
 $Comp
-L Device:LED D5
-U 1 1 61273E6B
-P 4700 4250
-F 0 "D5" V 4647 4330 50  0000 L CNN
-F 1 "LED_BL1" V 4738 4330 50  0000 L CNN
-F 2 "LED_THT:LED_D3.0mm" H 4700 4250 50  0001 C CNN
-F 3 "~" H 4700 4250 50  0001 C CNN
-F 4 "10mm" V 4700 4250 50  0001 C CNN "Montagehöhe"
-	1    4700 4250
-	0    -1   -1   0
-$EndComp
-$Comp
-L Device:LED D6
-U 1 1 612B359B
-P 5200 4250
-F 0 "D6" V 5147 4330 50  0000 L CNN
-F 1 "LED_BL2" V 5238 4330 50  0000 L CNN
-F 2 "LED_THT:LED_D3.0mm" H 5200 4250 50  0001 C CNN
-F 3 "~" H 5200 4250 50  0001 C CNN
-F 4 "10mm" V 5200 4250 50  0001 C CNN "Montagehöhe"
-	1    5200 4250
-	0    -1   -1   0
-$EndComp
-$Comp
-L Device:LED D7
-U 1 1 612F1FBB
-P 5700 4250
-F 0 "D7" V 5647 4330 50  0000 L CNN
-F 1 "LED_BL3" V 5738 4330 50  0000 L CNN
-F 2 "LED_THT:LED_D3.0mm" H 5700 4250 50  0001 C CNN
-F 3 "~" H 5700 4250 50  0001 C CNN
-F 4 "10mm" V 5700 4250 50  0001 C CNN "Montagehöhe"
-	1    5700 4250
-	0    -1   -1   0
-$EndComp
-$Comp
-L Device:LED D8
-U 1 1 61330C4E
-P 6200 4250
-F 0 "D8" V 6147 4330 50  0000 L CNN
-F 1 "LED_BL4" V 6238 4330 50  0000 L CNN
-F 2 "LED_THT:LED_D3.0mm" H 6200 4250 50  0001 C CNN
-F 3 "~" H 6200 4250 50  0001 C CNN
-F 4 "10mm" V 6200 4250 50  0001 C CNN "Montagehöhe"
-	1    6200 4250
-	0    -1   -1   0
-$EndComp
-$Comp
 L Device:LED D9
 U 1 1 6136FE41
@@
 F 1 "LED_BL5" V 6738 4330 50  0000 L CNN
 F 2 "LED_THT:LED_D3.0mm" H 6700 4250 50  0001 C CNN
-F 3 "~" H 6700 4250 50  0001 C CNN
+F 3 "http://www.qt-brightek.com/datasheet/QBL7IW60D-XX.pdf" H 6700 4250 50  0001 C CNN
 F 4 "10mm" V 6700 4250 50  0001 C CNN "Montagehöhe"
+F 5 "1516-QBL7IW60D-WW-ND" V 6700 4250 50  0001 C CNN "Digikey Part Number"
 	1    6700 4250
 	0    -1   -1   0
@@
 Text Notes 12550 3850 0    50   ~ 0
 KONSTANT\n
+$Comp
+L Device:LED D8
+U 1 1 6178E674
+P 6200 4250
+F 0 "D8" V 6147 4330 50  0000 L CNN
+F 1 "LED_BL4" V 6238 4330 50  0000 L CNN
+F 2 "LED_THT:LED_D3.0mm" H 6200 4250 50  0001 C CNN
+F 3 "http://www.qt-brightek.com/datasheet/QBL7IW60D-XX.pdf" H 6200 4250 50  0001 C CNN
+F 4 "10mm" V 6200 4250 50  0001 C CNN "Montagehöhe"
+F 5 "1516-QBL7IW60D-WW-ND" V 6200 4250 50  0001 C CNN "Digikey Part Number"
+	1    6200 4250
+	0    -1   -1   0
+$EndComp
+$Comp
+L Device:LED D7
+U 1 1 6178EE25
+P 5700 4250
+F 0 "D7" V 5647 4330 50  0000 L CNN
+F 1 "LED_BL3" V 5738 4330 50  0000 L CNN
+F 2 "LED_THT:LED_D3.0mm" H 5700 4250 50  0001 C CNN
+F 3 "http://www.qt-brightek.com/datasheet/QBL7IW60D-XX.pdf" H 5700 4250 50  0001 C CNN
+F 4 "10mm" V 5700 4250 50  0001 C CNN "Montagehöhe"
+F 5 "1516-QBL7IW60D-WW-ND" V 5700 4250 50  0001 C CNN "Digikey Part Number"
+	1    5700 4250
+	0    -1   -1   0
+$EndComp
+$Comp
+L Device:LED D6
+U 1 1 6178F54F
+P 5200 4250
+F 0 "D6" V 5147 4330 50  0000 L CNN
+F 1 "LED_BL2" V 5238 4330 50  0000 L CNN
+F 2 "LED_THT:LED_D3.0mm" H 5200 4250 50  0001 C CNN
+F 3 "http://www.qt-brightek.com/datasheet/QBL7IW60D-XX.pdf" H 5200 4250 50  0001 C CNN
+F 4 "10mm" V 5200 4250 50  0001 C CNN "Montagehöhe"
+F 5 "1516-QBL7IW60D-WW-ND" V 5200 4250 50  0001 C CNN "Digikey Part Number"
+	1    5200 4250
+	0    -1   -1   0
+$EndComp
+$Comp
+L Device:LED D5
+U 1 1 6178FF52
+P 4700 4250
+F 0 "D5" V 4647 4330 50  0000 L CNN
+F 1 "LED_BL1" V 4738 4330 50  0000 L CNN
+F 2 "LED_THT:LED_D3.0mm" H 4700 4250 50  0001 C CNN
+F 3 "http://www.qt-brightek.com/datasheet/QBL7IW60D-XX.pdf" H 4700 4250 50  0001 C CNN
+F 4 "10mm" V 4700 4250 50  0001 C CNN "Montagehöhe"
+F 5 "1516-QBL7IW60D-WW-ND" V 4700 4250 50  0001 C CNN "Digikey Part Number"
+	1    4700 4250
+	0    -1   -1   0
+$EndComp
 $EndSCHEMATC
