File: 7SegmentDriver.sch (KiCad schematic (older format))
At the start: 9 parts

Commit message: - Display Driving abgeschlossen
Parts:
- added C?: NA, Capacitor_SMD:C_0603_1608Metric, symbol Device:C
- added R?: 0R, Resistor_SMD:R_0603_1608Metric, symbol Device:R
- IC1, IC2, IC3, IC4: renamed from IC?; footprint SON50P300X300X63-11N -> TeKaDe:U-DFN3030-10
- U4: renamed from U?; value CD4514 -> CD4514BM
- U5: renamed from U?; value CD4511 -> CD4511BPWR; footprint Package_SO:SOIC-24W_7.5x15.4mm_P1.27mm -> Package_SO:TSSOP-14_4.4x5mm_P0.65mm
- gave numbers to parts that had none: 3
Connections:
- net BrightnessPWM: now also R?.2; no longer U5.4 (~BT)
- net GND: now also C?.2
- new net: C?.1, R?.1, U5.4 (~BT)
Other:
- note added: "RC Filter for PWM"
- note added: "Änderungen:\n- Bypass C für CD4511 / CD4514\n- Footprints hinzugefügt\n- Darlington Array Typ getauscht\n- optionaler RC Filter for PWM hinzugefuegt"
- note removed: "Änderungen:\n- Bypass C für CD4511 / CD4514"
- moved on the sheet: C41, U5

Commit message: - ATmega überarbeitet - Alle offenen Punkte zusammengefasst
Parts:
- gave numbers to parts that had none: 2
- renumbered C40 to C41, C41 to C43, J10 to J6, U4 to U7, U5 to U8

Commit message: - Platzoptimierungen
Parts:
- C41, C43: value 100n/10V/X7R -> 100n/16V/X7R; footprint Resistor_SMD:R_0603_1608Metric -> Capacitor_SMD:C_0402_1005Metric
- J6: value Conn_02x15_Odd_Even -> UIBoardCON2
Changed lines of the file:
@@
 AR Path="/60F87146/618C0CEF" Ref="J6"  Part="1"
 F 0 "J6" H 9750 4167 50  0000 C CNN
-F 1 "Conn_02x15_Odd_Even" H 9750 4076 50  0000 C CNN
+F 1 "UIBoardCON2" H 9750 4076 50  0000 C CNN
 F 2 "Connector_PinSocket_2.54mm:PinSocket_2x15_P2.54mm_Vertical" H 9700 3250 50  0001 C CNN
 F 3 "~" H 9700 3250 50  0001 C CNN
@@
 AR Path="/60F87146/6202C82F" Ref="C41"  Part="1"
 F 0 "C41" V 1050 5300 50  0000 L CNN
-F 1 "100n/10V/X7R" V 950 5100 50  0000 L CNN
-F 2 "Resistor_SMD:R_0603_1608Metric" H 838 5200 50  0001 C CNN
+F 1 "100n/16V/X7R" V 950 5100 50  0000 L CNN
+F 2 "Capacitor_SMD:C_0402_1005Metric" H 838 5200 50  0001 C CNN
 F 3 "~" H 800 5350 50  0001 C CNN
 	1    800  5350
@@
 AR Path="/60F87146/620341F4" Ref="C43"  Part="1"
 F 0 "C43" V 2450 1000 50  0000 L CNN
-F 1 "100n/10V/X7R" V 2350 800 50  0000 L CNN
-F 2 "Resistor_SMD:R_0603_1608Metric" H 2238 900 50  0001 C CNN
+F 1 "100n/16V/X7R" V 2350 800 50  0000 L CNN
+F 2 "Capacitor_SMD:C_0402_1005Metric" H 2238 900 50  0001 C CNN
 F 3 "~" H 2200 1050 50  0001 C CNN
 	1    2200 1050
