File: 7SegmentDriver.sch (KiCad schematic (older format))
At the start: 11 parts, among them IC1 ULN2003F12FN-7, IC2 ULN2003F12FN-7, IC3 ULN2003F12FN-7, IC4 ULN2003F12FN-7, J6 UIBoardCON2, U7 CD4514BM, U8 CD4511BPWR

Commit message: - Schaltbare BL Versorgung fertig - kleinere Value Anpassungen - Finale Annotation
Parts:
- renumbered C41 to C38, C42 to C39, C43 to C40, J6 to J10, R10 to R39, IC1 to U10, IC2 to U11, IC3 to U12, IC4 to U13, U7 to U8, U8 to U9

Commit message: - fix: footprint getauscht
Parts:
- U9: footprint Package_SO:TSSOP-14_4.4x5mm_P0.65mm -> Package_SO:TSSOP-16_4.4x5mm_P0.65mm
Changed lines of the file:
@@
 F 0 "U9" H 3500 2170 50  0000 C CNN
 F 1 "CD4511BPWR" H 3500 2079 50  0000 C CNN
-F 2 "Package_SO:TSSOP-14_4.4x5mm_P0.65mm" H 3500 1400 50  0001 L BNN
+F 2 "Package_SO:TSSOP-16_4.4x5mm_P0.65mm" H 3500 1400 50  0001 L BNN
 F 3 "60K5141" H 3500 1400 50  0001 L BNN
 F 4 "CD4511BE" H 3500 1400 50  0001 L BNN "Field4"

Commit message: - neue Stecker hinzugefügt, Annotation überall entsprechend angepasst Footprint fehlt noch
Parts:
- renumbered J10 to J6
Changed lines of the file:
@@
 P 9700 3250
 AR Path="/618C0CEF" Ref="J?"  Part="1"
-AR Path="/60F87146/618C0CEF" Ref="J10"  Part="1"
-F 0 "J10" H 9750 4167 50  0000 C CNN
+AR Path="/60F87146/618C0CEF" Ref="J6"  Part="1"
+F 0 "J6" H 9750 4167 50  0000 C CNN
 F 1 "UIBoardCON2" H 9750 4076 50  0000 C CNN
 F 2 "Connector_PinSocket_2.54mm:PinSocket_2x15_P2.54mm_Vertical" H 9700 3250 50  0001 C CNN

Commit message: - Layout Zwischenstand, UI Board Ansteuerung fast fertig - GPIOs von ATmega komplett umsortiert - Darlington Anschlüsse umsortiert
Connections:
- net CathodeDigit1: now also U12.7 (OUT4); no longer U10.8 (OUT3)
- net CathodeDigit10: now also U10.7 (OUT4); no longer U12.7 (OUT4)
- net CathodeDigit10Signal: now also U10.4 (IN4); no longer U12.4 (IN4)
- net CathodeDigit11: now also U11.8 (OUT3); no longer U13.10 (OUT1)
- net CathodeDigit11Signal: now also U11.3 (IN3); no longer U13.1 (IN1)
- net CathodeDigit12: now also U11.9 (OUT2); no longer U13.9 (OUT2)
- net CathodeDigit12Signal: now also U11.2 (IN2); no longer U13.2 (IN2)
- net CathodeDigit13: now also U12.10 (OUT1); no longer U13.8 (OUT3)
- net CathodeDigit13Signal: now also U12.1 (IN1); no longer U13.3 (IN3)
- net CathodeDigit14: now also U10.10 (OUT1); no longer U13.7 (OUT4)
- net CathodeDigit14Signal: now also U10.1 (IN1); no longer U13.4 (IN4)
- net CathodeDigit1Signal: now also U12.4 (IN4); no longer U10.3 (IN3)
- net CathodeDigit2: now also U13.10 (OUT1); no longer U10.7 (OUT4)
- net CathodeDigit2Signal: now also U13.1 (IN1); no longer U10.4 (IN4)
- net CathodeDigit3: now also U13.9 (OUT2); no longer U11.10 (OUT1)
- net CathodeDigit3Signal: now also U13.2 (IN2); no longer U11.1 (IN1)
- net CathodeDigit4: now also U13.8 (OUT3); no longer U11.9 (OUT2)
- net CathodeDigit4Signal: now also U13.3 (IN3); no longer U11.2 (IN2)
- net CathodeDigit5: now also U13.7 (OUT4); no longer U11.8 (OUT3)
- net CathodeDigit5Signal: now also U13.4 (IN4); no longer U11.3 (IN3)
- net CathodeDigit7: now also U10.8 (OUT3); no longer U12.10 (OUT1)
- net CathodeDigit7Signal: now also U10.3 (IN3); no longer U12.1 (IN1)
- net CathodeDigit8: now also U10.9 (OUT2); no longer U12.9 (OUT2)
- net CathodeDigit8Signal: now also U10.2 (IN2); no longer U12.2 (IN2)
- net CathodeDigit9: now also U11.10 (OUT1); no longer U12.8 (OUT3)
- net CathodeDigit9Signal: now also U11.1 (IN1); no longer U12.3 (IN3)
- net CathodeDigitA: now also U12.9 (OUT2); no longer U10.10 (OUT1)
- net CathodeDigitASignal: now also U12.2 (IN2); no longer U10.1 (IN1)
- net CathodeDigitB: now also U12.8 (OUT3); no longer U10.9 (OUT2)
- net CathodeDigitBSignal: now also U12.3 (IN3); no longer U10.2 (IN2)
Changed lines of the file:
@@
 Text HLabel 1250 4300 0    50   Input ~ 0
 7Seg_Decoder_D1
-Text Label 6850 3750 0    50   ~ 0
+Text Label 6850 6450 0    50   ~ 0
 CathodeDigit5
-Text Label 6850 3650 0    50   ~ 0
+Text Label 6850 6350 0    50   ~ 0
 CathodeDigit4
-Text Label 6850 3550 0    50   ~ 0
+Text Label 6850 6250 0    50   ~ 0
 CathodeDigit3
-Text Label 6850 2550 0    50   ~ 0
+Text Label 6850 6150 0    50   ~ 0
 CathodeDigit2
-Text Label 6850 2450 0    50   ~ 0
+Text Label 6850 5150 0    50   ~ 0
 CathodeDigit1
-Text Label 6850 2350 0    50   ~ 0
+Text Label 6850 5050 0    50   ~ 0
 CathodeDigitB
-Text Label 6850 2250 0    50   ~ 0
-CathodeDigitA
 Text Label 6850 3850 0    50   ~ 0
 CathodeDigit6
-Text Label 6850 5150 0    50   ~ 0
+Text Label 6850 2550 0    50   ~ 0
 CathodeDigit10
-Text Label 6850 5050 0    50   ~ 0
+Text Label 6850 3550 0    50   ~ 0
 CathodeDigit9
-Text Label 6850 4950 0    50   ~ 0
+Text Label 6850 2350 0    50   ~ 0
 CathodeDigit8
+Text Label 6850 2450 0    50   ~ 0
+CathodeDigit7
+Text Label 6850 3650 0    50   ~ 0
+CathodeDigit12
+Text Label 6850 3750 0    50   ~ 0
+CathodeDigit11
 Text Label 6850 4850 0    50   ~ 0
-CathodeDigit7
-Text Label 6850 6250 0    50   ~ 0
-CathodeDigit12
-Text Label 6850 6150 0    50   ~ 0
-CathodeDigit11
-Text Label 6850 6350 0    50   ~ 0
 CathodeDigit13
-Text Label 6850 6450 0    50   ~ 0
+Text Label 6850 2250 0    50   ~ 0
 CathodeDigit14
-Text Label 5350 6150 2    50   ~ 0
+Text Label 5350 3750 2    50   ~ 0
 CathodeDigit11Signal
-Text Label 5350 6250 2    50   ~ 0
+Text Label 5350 3650 2    50   ~ 0
 CathodeDigit12Signal
-Text Label 5350 5050 2    50   ~ 0
+Text Label 5350 3550 2    50   ~ 0
 CathodeDigit9Signal
-Text Label 5350 5150 2    50   ~ 0
+Text Label 5350 2550 2    50   ~ 0
 CathodeDigit10Signal
-Text Label 5350 4850 2    50   ~ 0
+Text Label 5350 2450 2    50   ~ 0
 CathodeDigit7Signal
-Text Label 5350 4950 2    50   ~ 0
+Text Label 5350 2350 2    50   ~ 0
 CathodeDigit8Signal
 $Comp
@@
 	1    0    0    -1
 $EndComp
-Text Label 5350 3750 2    50   ~ 0
+Text Label 5350 6450 2    50   ~ 0
 CathodeDigit5Signal
-Text Label 5350 3650 2    50   ~ 0
+Text Label 5350 6350 2    50   ~ 0
 CathodeDigit4Signal
-Text Label 5350 3550 2    50   ~ 0
+Text Label 5350 6250 2    50   ~ 0
 CathodeDigit3Signal
-Text Label 5350 2550 2    50   ~ 0
+Text Label 5350 6150 2    50   ~ 0
 CathodeDigit2Signal
-Text Label 5350 2450 2    50   ~ 0
+Text Label 5350 5150 2    50   ~ 0
 CathodeDigit1Signal
-Text Label 5350 2350 2    50   ~ 0
+Text Label 5350 5050 2    50   ~ 0
 CathodeDigitBSignal
-Text Label 5350 2250 2    50   ~ 0
+Text Label 5350 4950 2    50   ~ 0
 CathodeDigitASignal
 Wire Wire Line
-	5350 3750 5500 3750
-Wire Wire Line
-	5500 3650 5350 3650
-Wire Wire Line
-	5350 3550 5500 3550
-Wire Wire Line
-	5500 2550 5350 2550
+	5350 6450 5500 6450
+Wire Wire Line
+	5500 6350 5350 6350
+Wire Wire Line
+	5350 6250 5500 6250
+Wire Wire Line
+	5500 6150 5350 6150
+Wire Wire Line
+	5350 5150 5500 5150
+Wire Wire Line
+	5350 5050 5500 5050
+Wire Wire Line
+	5350 4950 5500 4950
+Wire Wire Line
+	5350 3650 5500 3650
+Wire Wire Line
+	5500 3750 5350 3750
+Wire Wire Line
+	5350 2550 5500 2550
+Wire Wire Line
+	5500 3550 5350 3550
+Wire Wire Line
+	5350 2350 5500 2350
 Wire Wire Line
 	5350 2450 5500 2450
-Wire Wire Line
-	5350 2350 5500 2350
-Wire Wire Line
-	5350 2250 5500 2250
-Wire Wire Line
-	5350 6250 5500 6250
-Wire Wire Line
-	5500 6150 5350 6150
-Wire Wire Line
-	5350 5150 5500 5150
-Wire Wire Line
-	5500 5050 5350 5050
-Wire Wire Line
-	5350 4950 5500 4950
-Wire Wire Line
-	5350 4850 5500 4850
 Wire Wire Line
 	5350 3850 5500 3850
 Text Label 5350 3850 2    50   ~ 0
 CathodeDigit6Signal
-Text Label 5350 6350 2    50   ~ 0
+Text Label 5350 4850 2    50   ~ 0
 CathodeDigit13Signal
-Text Label 5350 6450 2    50   ~ 0
+Text Label 5350 2250 2    50   ~ 0
 CathodeDigit14Signal
 $Comp
@@
 $EndComp
 Wire Wire Line
-	5350 6350 5500 6350
-Wire Wire Line
-	5500 6450 5350 6450
-Wire Wire Line
-	6700 6250 6850 6250
-Wire Wire Line
-	6850 6150 6700 6150
-Wire Wire Line
-	6700 6350 6850 6350
-Wire Wire Line
-	6850 6450 6700 6450
+	5350 4850 5500 4850
+Wire Wire Line
+	5500 2250 5350 2250
+Wire Wire Line
+	6700 3650 6850 3650
+Wire Wire Line
+	6850 3750 6700 3750
+Wire Wire Line
+	6700 4850 6850 4850
+Wire Wire Line
+	6850 2250 6700 2250
 Wire Wire Line
 	6700 6550 6750 6550
@@
 $EndComp
 Wire Wire Line
-	6700 2350 6850 2350
-Wire Wire Line
-	6850 2250 6700 2250
-Wire Wire Line
-	6700 2450 6850 2450
-Wire Wire Line
-	6850 2550 6700 2550
+	6700 5050 6850 5050
+Wire Wire Line
+	6850 6150 6700 6150
 Wire Wire Line
 	6700 2650 6750 2650
@@
 $EndComp
 Wire Wire Line
-	6700 3650 6850 3650
-Wire Wire Line
-	6850 3550 6700 3550
-Wire Wire Line
-	6700 3750 6850 3750
+	6700 6350 6850 6350
+Wire Wire Line
+	6850 6250 6700 6250
+Wire Wire Line
+	6700 6450 6850 6450
 Wire Wire Line
 	6850 3850 6700 3850
@@
 $EndComp
 Wire Wire Line
-	6700 4950 6850 4950
-Wire Wire Line
-	6850 4850 6700 4850
-Wire Wire Line
-	6700 5050 6850 5050
-Wire Wire Line
-	6850 5150 6700 5150
+	6700 2350 6850 2350
+Wire Wire Line
+	6850 2450 6700 2450
+Wire Wire Line
+	6700 3550 6850 3550
+Wire Wire Line
+	6850 2550 6700 2550
 Wire Wire Line
 	6700 5250 6750 5250
-Wire Wire Line
-	6750 5250 6750 4500
 Wire Wire Line
 	5450 5250 5500 5250
@@
 NoConn ~ 9500 3850
 NoConn ~ 9500 3950
+Wire Wire Line
+	6700 5150 6850 5150
+Wire Wire Line
+	6750 5250 6750 4500
+Wire Wire Line
+	6850 4950 6700 4950
+Text Label 6850 4950 0    50   ~ 0
+CathodeDigitA
 $EndSCHEMATC

Commit message: - merged Fix pad not on gnd
Changed lines of the file:
@@
-	1    0    0    -1
-$EndComp
-$Comp
-L power:GND #PWR0109
-U 1 1 60FC7F2E
-P 6100 3000
-F 0 "#PWR0109" H 6100 2750 50  0001 C CNN
-F 1 "GND" H 6105 2827 50  0000 C CNN
-F 2 "" H 6100 3000 50  0001 C CNN
-F 3 "" H 6100 3000 50  0001 C CNN
-	1    6100 3000
 	1    0    0    -1
 $EndComp
@@
 	1    0    0    -1
 $EndComp
-$Comp
-L power:GND #PWR0110
-U 1 1 6107D228
-P 6100 4300
-F 0 "#PWR0110" H 6100 4050 50  0001 C CNN
-F 1 "GND" H 6105 4127 50  0000 C CNN
-F 2 "" H 6100 4300 50  0001 C CNN
-F 3 "" H 6100 4300 50  0001 C CNN
-	1    6100 4300
-	1    0    0    -1
-$EndComp
 Wire Wire Line
 	5450 4300 5450 3950
-Wire Wire Line
-	6100 4300 6100 4250
 $Comp
 L power:+5V #PWR?
@@
 	1    0    0    -1
 $EndComp
-$Comp
-L power:GND #PWR0111
-U 1 1 6108D326
-P 6100 5600
-F 0 "#PWR0111" H 6100 5350 50  0001 C CNN
-F 1 "GND" H 6105 5427 50  0000 C CNN
-F 2 "" H 6100 5600 50  0001 C CNN
-F 3 "" H 6100 5600 50  0001 C CNN
-	1    6100 5600
-	1    0    0    -1
-$EndComp
 Wire Wire Line
 	5450 5600 5450 5250
-Wire Wire Line
-	6100 5600 6100 5550
 Wire Wire Line
 	6750 3200 6750 3950
@@
 	1    0    0    -1
 $EndComp
-$Comp
-L power:GND #PWR0112
-U 1 1 610F2AFB
-P 6100 6900
-F 0 "#PWR0112" H 6100 6650 50  0001 C CNN
-F 1 "GND" H 6105 6727 50  0000 C CNN
-F 2 "" H 6100 6900 50  0001 C CNN
-F 3 "" H 6100 6900 50  0001 C CNN
-	1    6100 6900
-	1    0    0    -1
-$EndComp
 Wire Wire Line
 	5450 6900 5450 6550
-Wire Wire Line
-	6100 6900 6100 6850
-Wire Wire Line
-	6100 2950 6100 3000
 $Comp
 L Device:R R39
