File: LevelShift.sch (KiCad schematic (older format))
At the start: 6 parts, among them U19 SN74LV1T126, U20 SN74LV1T126, U21 SN74LV1T126

Commit message: - ATmega überarbeitet - Alle offenen Punkte zusammengefasst
Parts:
- renumbered C80 to C7, C81 to C8, C82 to C9, U21 to U3, U19 to U4, U20 to U5
Changed lines of the file:
@@
 $Descr A4 11693 8268
 encoding utf-8
-Sheet 6 9
+Sheet 4 9
 Title ""
 Date ""
@@
 P 5550 5400
 AR Path="/61321836" Ref="U?"  Part="1"
-AR Path="/6131300C/61321836" Ref="U20"  Part="1"
-F 0 "U20" H 5550 5725 50  0000 C CNN
+AR Path="/6131300C/61321836" Ref="U5"  Part="1"
+F 0 "U5" H 5550 5725 50  0000 C CNN
 F 1 "SN74LV1T126" H 5550 5634 50  0000 C CNN
 F 2 "Package_TO_SOT_SMD:SOT-23-5" H 5550 5150 50  0001 C CNN
@@
 AR Path="/60D33366/6132183C" Ref="#PWR?"  Part="1"
 AR Path="/6132183C" Ref="#PWR?"  Part="1"
-AR Path="/6131300C/6132183C" Ref="#PWR0180"  Part="1"
-F 0 "#PWR0180" H 6250 5450 50  0001 C CNN
+AR Path="/6131300C/6132183C" Ref="#PWR033"  Part="1"
+F 0 "#PWR033" H 6250 5450 50  0001 C CNN
 F 1 "GND" H 6255 5527 50  0000 C CNN
 F 2 "" H 6250 5700 50  0001 C CNN
@@
 AR Path="/60D33366/61321843" Ref="C?"  Part="1"
 AR Path="/61321843" Ref="C?"  Part="1"
-AR Path="/6131300C/61321843" Ref="C82"  Part="1"
-F 0 "C82" V 6500 5150 50  0000 L CNN
+AR Path="/6131300C/61321843" Ref="C9"  Part="1"
+F 0 "C9" V 6500 5150 50  0000 L CNN
 F 1 "100n/10V/X7R" V 6400 4950 50  0000 L CNN
 F 2 "Resistor_SMD:R_0603_1608Metric" H 6288 5050 50  0001 C CNN
@@
 AR Path="/60D33366/61321849" Ref="#PWR?"  Part="1"
 AR Path="/61321849" Ref="#PWR?"  Part="1"
-AR Path="/6131300C/61321849" Ref="#PWR0181"  Part="1"
-F 0 "#PWR0181" H 5100 5450 50  0001 C CNN
+AR Path="/6131300C/61321849" Ref="#PWR024"  Part="1"
+F 0 "#PWR024" H 5100 5450 50  0001 C CNN
 F 1 "GND" H 5105 5527 50  0000 C CNN
 F 2 "" H 5100 5700 50  0001 C CNN
@@
 P 5100 5050
 AR Path="/61321851" Ref="#PWR?"  Part="1"
-AR Path="/6131300C/61321851" Ref="#PWR0182"  Part="1"
-F 0 "#PWR0182" H 5100 4900 50  0001 C CNN
+AR Path="/6131300C/61321851" Ref="#PWR023"  Part="1"
+F 0 "#PWR023" H 5100 4900 50  0001 C CNN
 F 1 "+5V" H 5115 5223 50  0000 C CNN
 F 2 "" H 5100 5050 50  0001 C CNN
@@
 AR Path="/620639FD/6132185B" Ref="#PWR?"  Part="1"
 AR Path="/6132185B" Ref="#PWR?"  Part="1"
-AR Path="/6131300C/6132185B" Ref="#PWR0183"  Part="1"
-F 0 "#PWR0183" H 6000 4900 50  0001 C CNN
+AR Path="/6131300C/6132185B" Ref="#PWR027"  Part="1"
+F 0 "#PWR027" H 6000 4900 50  0001 C CNN
 F 1 "+3.3V" H 6015 5223 50  0000 C CNN
 F 2 "" H 6000 5050 50  0001 C CNN
@@
 AR Path="/620639FD/61321865" Ref="#PWR?"  Part="1"
 AR Path="/61321865" Ref="#PWR?"  Part="1"
-AR Path="/6131300C/61321865" Ref="#PWR0184"  Part="1"
-F 0 "#PWR0184" H 6250 4900 50  0001 C CNN
+AR Path="/6131300C/61321865" Ref="#PWR032"  Part="1"
+F 0 "#PWR032" H 6250 4900 50  0001 C CNN
 F 1 "+3.3V" H 6265 5223 50  0000 C CNN
 F 2 "" H 6250 5050 50  0001 C CNN
@@
 P 5550 3750
 AR Path="/61348F64" Ref="U?"  Part="1"
-AR Path="/6131300C/61348F64" Ref="U19"  Part="1"
-F 0 "U19" H 5550 4075 50  0000 C CNN
+AR Path="/6131300C/61348F64" Ref="U4"  Part="1"
+F 0 "U4" H 5550 4075 50  0000 C CNN
 F 1 "SN74LV1T126" H 5550 3984 50  0000 C CNN
 F 2 "Package_TO_SOT_SMD:SOT-23-5" H 5550 3500 50  0001 C CNN
@@
 AR Path="/60D33366/61348F6E" Ref="#PWR?"  Part="1"
 AR Path="/61348F6E" Ref="#PWR?"  Part="1"
-AR Path="/6131300C/61348F6E" Ref="#PWR0185"  Part="1"
-F 0 "#PWR0185" H 6250 3800 50  0001 C CNN
+AR Path="/6131300C/61348F6E" Ref="#PWR031"  Part="1"
+F 0 "#PWR031" H 6250 3800 50  0001 C CNN
 F 1 "GND" H 6255 3877 50  0000 C CNN
 F 2 "" H 6250 4050 50  0001 C CNN
@@
 AR Path="/60D33366/61348F79" Ref="C?"  Part="1"
 AR Path="/61348F79" Ref="C?"  Part="1"
-AR Path="/6131300C/61348F79" Ref="C81"  Part="1"
-F 0 "C81" V 6500 3500 50  0000 L CNN
+AR Path="/6131300C/61348F79" Ref="C8"  Part="1"
+F 0 "C8" V 6500 3500 50  0000 L CNN
 F 1 "100n/10V/X7R" V 6400 3300 50  0000 L CNN
 F 2 "Resistor_SMD:R_0603_1608Metric" H 6288 3400 50  0001 C CNN
@@
 AR Path="/60D33366/61348F83" Ref="#PWR?"  Part="1"
 AR Path="/61348F83" Ref="#PWR?"  Part="1"
-AR Path="/6131300C/61348F83" Ref="#PWR0186"  Part="1"
-F 0 "#PWR0186" H 5100 3800 50  0001 C CNN
+AR Path="/6131300C/61348F83" Ref="#PWR022"  Part="1"
+F 0 "#PWR022" H 5100 3800 50  0001 C CNN
 F 1 "GND" H 5105 3877 50  0000 C CNN
 F 2 "" H 5100 4050 50  0001 C CNN
@@
 P 5100 3400
 AR Path="/61348F8F" Ref="#PWR?"  Part="1"
-AR Path="/6131300C/61348F8F" Ref="#PWR0187"  Part="1"
-F 0 "#PWR0187" H 5100 3250 50  0001 C CNN
+AR Path="/6131300C/61348F8F" Ref="#PWR021"  Part="1"
+F 0 "#PWR021" H 5100 3250 50  0001 C CNN
 F 1 "+5V" H 5115 3573 50  0000 C CNN
 F 2 "" H 5100 3400 50  0001 C CNN
@@
 AR Path="/620639FD/61348F9C" Ref="#PWR?"  Part="1"
 AR Path="/61348F9C" Ref="#PWR?"  Part="1"
-AR Path="/6131300C/61348F9C" Ref="#PWR0188"  Part="1"
-F 0 "#PWR0188" H 6000 3250 50  0001 C CNN
+AR Path="/6131300C/61348F9C" Ref="#PWR026"  Part="1"
+F 0 "#PWR026" H 6000 3250 50  0001 C CNN
 F 1 "+3.3V" H 6015 3573 50  0000 C CNN
 F 2 "" H 6000 3400 50  0001 C CNN
@@
 AR Path="/620639FD/61348FA9" Ref="#PWR?"  Part="1"
 AR Path="/61348FA9" Ref="#PWR?"  Part="1"
-AR Path="/6131300C/61348FA9" Ref="#PWR0189"  Part="1"
-F 0 "#PWR0189" H 6250 3250 50  0001 C CNN
+AR Path="/6131300C/61348FA9" Ref="#PWR030"  Part="1"
+F 0 "#PWR030" H 6250 3250 50  0001 C CNN
 F 1 "+3.3V" H 6265 3573 50  0000 C CNN
 F 2 "" H 6250 3400 50  0001 C CNN
@@
 AR Path="/620639FD/6132182C" Ref="#PWR?"  Part="1"
 AR Path="/6132182C" Ref="#PWR?"  Part="1"
-AR Path="/6131300C/6132182C" Ref="#PWR0179"  Part="1"
-F 0 "#PWR0179" H 5100 2050 50  0001 C CNN
+AR Path="/6131300C/6132182C" Ref="#PWR019"  Part="1"
+F 0 "#PWR019" H 5100 2050 50  0001 C CNN
 F 1 "+3.3V" H 5115 2373 50  0000 C CNN
 F 2 "" H 5100 2200 50  0001 C CNN
@@
 P 6250 2200
 AR Path="/61321822" Ref="#PWR?"  Part="1"
-AR Path="/6131300C/61321822" Ref="#PWR0178"  Part="1"
-F 0 "#PWR0178" H 6250 2050 50  0001 C CNN
+AR Path="/6131300C/61321822" Ref="#PWR028"  Part="1"
+F 0 "#PWR028" H 6250 2050 50  0001 C CNN
 F 1 "+5V" H 6265 2373 50  0000 C CNN
 F 2 "" H 6250 2200 50  0001 C CNN
@@
 P 6000 2200
 AR Path="/6132181C" Ref="#PWR?"  Part="1"
-AR Path="/6131300C/6132181C" Ref="#PWR0177"  Part="1"
-F 0 "#PWR0177" H 6000 2050 50  0001 C CNN
+AR Path="/6131300C/6132181C" Ref="#PWR025"  Part="1"
+F 0 "#PWR025" H 6000 2050 50  0001 C CNN
 F 1 "+5V" H 6015 2373 50  0000 C CNN
 F 2 "" H 6000 2200 50  0001 C CNN
@@
 AR Path="/60D33366/61321814" Ref="#PWR?"  Part="1"
 AR Path="/61321814" Ref="#PWR?"  Part="1"
-AR Path="/6131300C/61321814" Ref="#PWR0176"  Part="1"
-F 0 "#PWR0176" H 5100 2600 50  0001 C CNN
+AR Path="/6131300C/61321814" Ref="#PWR020"  Part="1"
+F 0 "#PWR020" H 5100 2600 50  0001 C CNN
 F 1 "GND" H 5105 2677 50  0000 C CNN
 F 2 "" H 5100 2850 50  0001 C CNN
@@
 AR Path="/60D33366/6132180E" Ref="C?"  Part="1"
 AR Path="/6132180E" Ref="C?"  Part="1"
-AR Path="/6131300C/6132180E" Ref="C80"  Part="1"
-F 0 "C80" V 6500 2300 50  0000 L CNN
+AR Path="/6131300C/6132180E" Ref="C7"  Part="1"
+F 0 "C7" V 6500 2300 50  0000 L CNN
 F 1 "100n/10V/X7R" V 6400 2100 50  0000 L CNN
 F 2 "Resistor_SMD:R_0603_1608Metric" H 6288 2200 50  0001 C CNN
@@
 AR Path="/60D33366/61321807" Ref="#PWR?"  Part="1"
 AR Path="/61321807" Ref="#PWR?"  Part="1"
-AR Path="/6131300C/61321807" Ref="#PWR0175"  Part="1"
-F 0 "#PWR0175" H 6250 2600 50  0001 C CNN
+AR Path="/6131300C/61321807" Ref="#PWR029"  Part="1"
+F 0 "#PWR029" H 6250 2600 50  0001 C CNN
 F 1 "GND" H 6255 2677 50  0000 C CNN
 F 2 "" H 6250 2850 50  0001 C CNN
@@
 P 5550 2550
 AR Path="/61321801" Ref="U?"  Part="1"
-AR Path="/6131300C/61321801" Ref="U21"  Part="1"
-F 0 "U21" H 5550 2875 50  0000 C CNN
+AR Path="/6131300C/61321801" Ref="U3"  Part="1"
+F 0 "U3" H 5550 2875 50  0000 C CNN
 F 1 "SN74LV1T126" H 5550 2784 50  0000 C CNN
 F 2 "Package_TO_SOT_SMD:SOT-23-5" H 5550 2300 50  0001 C CNN

Commit message: - Platzoptimierungen
Parts:
- C7, C8, C9: value 100n/10V/X7R -> 100n/16V/X7R; footprint Resistor_SMD:R_0603_1608Metric -> Capacitor_SMD:C_0402_1005Metric
Changed lines of the file:
@@
 AR Path="/6131300C/61321843" Ref="C9"  Part="1"
 F 0 "C9" V 6500 5150 50  0000 L CNN
-F 1 "100n/10V/X7R" V 6400 4950 50  0000 L CNN
-F 2 "Resistor_SMD:R_0603_1608Metric" H 6288 5050 50  0001 C CNN
+F 1 "100n/16V/X7R" V 6400 4950 50  0000 L CNN
+F 2 "Capacitor_SMD:C_0402_1005Metric" H 6288 5050 50  0001 C CNN
 F 3 "~" H 6250 5200 50  0001 C CNN
 	1    6250 5200
@@
 AR Path="/6131300C/61348F79" Ref="C8"  Part="1"
 F 0 "C8" V 6500 3500 50  0000 L CNN
-F 1 "100n/10V/X7R" V 6400 3300 50  0000 L CNN
-F 2 "Resistor_SMD:R_0603_1608Metric" H 6288 3400 50  0001 C CNN
+F 1 "100n/16V/X7R" V 6400 3300 50  0000 L CNN
+F 2 "Capacitor_SMD:C_0402_1005Metric" H 6288 3400 50  0001 C CNN
 F 3 "~" H 6250 3550 50  0001 C CNN
 	1    6250 3550
@@
 AR Path="/6131300C/6132180E" Ref="C7"  Part="1"
 F 0 "C7" V 6500 2300 50  0000 L CNN
-F 1 "100n/10V/X7R" V 6400 2100 50  0000 L CNN
-F 2 "Resistor_SMD:R_0603_1608Metric" H 6288 2200 50  0001 C CNN
+F 1 "100n/16V/X7R" V 6400 2100 50  0000 L CNN
+F 2 "Capacitor_SMD:C_0402_1005Metric" H 6288 2200 50  0001 C CNN
 F 3 "~" H 6250 2350 50  0001 C CNN
 	1    6250 2350

Commit message: [fix:] general troublespots -> notes
Parts:
- removed C9: 100n/16V/X7R, Capacitor_SMD:C_0402_1005Metric, symbol Device:C
- removed U5: SN74LV1T126, Package_TO_SOT_SMD:SOT-23-5, symbol TeKaDe:SN74LV1T126
Other:
- note removed: "Converts 5V RUN Signal from ATMega to 3V3 for RPI"
Changed lines of the file:
@@
 $Descr A4 11693 8268
 encoding utf-8
-Sheet 4 9
+Sheet 7 9
 Title ""
 Date ""
@@
 Comment4 ""
 $EndDescr
-$Comp
-L TeKaDe:SN74LV1T126 U?
-U 1 1 61321836
-P 5550 5400
-AR Path="/61321836" Ref="U?"  Part="1"
-AR Path="/6131300C/61321836" Ref="U5"  Part="1"
-F 0 "U5" H 5550 5725 50  0000 C CNN
-F 1 "SN74LV1T126" H 5550 5634 50  0000 C CNN
-F 2 "Package_TO_SOT_SMD:SOT-23-5" H 5550 5150 50  0001 C CNN
-F 3 "" H 5350 5350 50  0001 C CNN
-	1    5550 5400
-	1    0    0    -1
-$EndComp
-$Comp
-L power:GND #PWR?
-U 1 1 6132183C
-P 6250 5700
-AR Path="/60D33366/6132183C" Ref="#PWR?"  Part="1"
-AR Path="/6132183C" Ref="#PWR?"  Part="1"
-AR Path="/6131300C/6132183C" Ref="#PWR033"  Part="1"
-F 0 "#PWR033" H 6250 5450 50  0001 C CNN
-F 1 "GND" H 6255 5527 50  0000 C CNN
-F 2 "" H 6250 5700 50  0001 C CNN
-F 3 "" H 6250 5700 50  0001 C CNN
-	1    6250 5700
-	1    0    0    -1
-$EndComp
-Wire Wire Line
-	6250 5350 6250 5700
-$Comp
-L Device:C C?
-U 1 1 61321843
-P 6250 5200
-AR Path="/60D33366/61321843" Ref="C?"  Part="1"
-AR Path="/61321843" Ref="C?"  Part="1"
-AR Path="/6131300C/61321843" Ref="C9"  Part="1"
-F 0 "C9" V 6500 5150 50  0000 L CNN
-F 1 "100n/16V/X7R" V 6400 4950 50  0000 L CNN
-F 2 "Capacitor_SMD:C_0402_1005Metric" H 6288 5050 50  0001 C CNN
-F 3 "~" H 6250 5200 50  0001 C CNN
-	1    6250 5200
-	1    0    0    -1
-$EndComp
-$Comp
-L power:GND #PWR?
-U 1 1 61321849
-P 5100 5700
-AR Path="/60D33366/61321849" Ref="#PWR?"  Part="1"
-AR Path="/61321849" Ref="#PWR?"  Part="1"
-AR Path="/6131300C/61321849" Ref="#PWR024"  Part="1"
-F 0 "#PWR024" H 5100 5450 50  0001 C CNN
-F 1 "GND" H 5105 5527 50  0000 C CNN
-F 2 "" H 5100 5700 50  0001 C CNN
-F 3 "" H 5100 5700 50  0001 C CNN
-	1    5100 5700
-	1    0    0    -1
-$EndComp
-Wire Wire Line
-	5200 5500 5100 5500
-Wire Wire Line
-	5100 5500 5100 5700
-$Comp
-L power:+5V #PWR?
-U 1 1 61321851
-P 5100 5050
-AR Path="/61321851" Ref="#PWR?"  Part="1"
-AR Path="/6131300C/61321851" Ref="#PWR023"  Part="1"
-F 0 "#PWR023" H 5100 4900 50  0001 C CNN
-F 1 "+5V" H 5115 5223 50  0000 C CNN
-F 2 "" H 5100 5050 50  0001 C CNN
-F 3 "" H 5100 5050 50  0001 C CNN
-	1    5100 5050
-	1    0    0    -1
-$EndComp
-Wire Wire Line
-	5900 5500 7700 5500
-Wire Wire Line
-	5900 5300 6000 5300
-Wire Wire Line
-	6000 5300 6000 5050
-$Comp
-L power:+3.3V #PWR?
-U 1 1 6132185B
-P 6000 5050
-AR Path="/620639FD/6132185B" Ref="#PWR?"  Part="1"
-AR Path="/6132185B" Ref="#PWR?"  Part="1"
-AR Path="/6131300C/6132185B" Ref="#PWR027"  Part="1"
-F 0 "#PWR027" H 6000 4900 50  0001 C CNN
-F 1 "+3.3V" H 6015 5223 50  0000 C CNN
-F 2 "" H 6000 5050 50  0001 C CNN
-F 3 "" H 6000 5050 50  0001 C CNN
-	1    6000 5050
-	1    0    0    -1
-$EndComp
-Wire Wire Line
-	5100 5050 5100 5300
-Wire Wire Line
-	5100 5300 5200 5300
-Wire Wire Line
-	5200 5400 3500 5400
-$Comp
-L power:+3.3V #PWR?
-U 1 1 61321865
-P 6250 5050
-AR Path="/620639FD/61321865" Ref="#PWR?"  Part="1"
-AR Path="/61321865" Ref="#PWR?"  Part="1"
-AR Path="/6131300C/61321865" Ref="#PWR032"  Part="1"
-F 0 "#PWR032" H 6250 4900 50  0001 C CNN
-F 1 "+3.3V" H 6265 5223 50  0000 C CNN
-F 2 "" H 6250 5050 50  0001 C CNN
-F 3 "" H 6250 5050 50  0001 C CNN
-	1    6250 5050
-	1    0    0    -1
-$EndComp
-Text HLabel 7700 5500 2    50   Output ~ 0
-RUN_3V3
 $Comp
 L TeKaDe:SN74LV1T126 U?
@@
 	7650 3850 5900 3850
 Wire Notes Line
-	8450 4550 2950 4550
-Wire Notes Line
-	2950 4550 2950 6050
-Wire Notes Line
-	2950 6050 8450 6050
-Wire Notes Line
-	8450 6050 8450 4550
-Text Notes 3050 4700 0    50   ~ 0
-Converts 5V RUN Signal from ATMega to 3V3 for RPI
-Wire Notes Line
 	2950 1700 8450 1700
 Wire Notes Line
@@
 Text Notes 3050 1850 0    50   ~ 0
 Converts 5V UART from ATMega to 3V3 for RPI
-Text HLabel 3500 5400 0    50   Input ~ 0
-RUN_5V
 Text HLabel 7650 3850 2    50   Output ~ 0
 UART_TX_3V3

Commit message: - Schaltbare BL Versorgung fertig - kleinere Value Anpassungen - Finale Annotation
Parts:
- renumbered C7 to C71, C8 to C72, U3 to U15, U4 to U16
Changed lines of the file:
@@
 P 5550 3750
 AR Path="/61348F64" Ref="U?"  Part="1"
-AR Path="/6131300C/61348F64" Ref="U4"  Part="1"
-F 0 "U4" H 5550 4075 50  0000 C CNN
+AR Path="/6131300C/61348F64" Ref="U16"  Part="1"
+F 0 "U16" H 5550 4075 50  0000 C CNN
 F 1 "SN74LV1T126" H 5550 3984 50  0000 C CNN
 F 2 "Package_TO_SOT_SMD:SOT-23-5" H 5550 3500 50  0001 C CNN
@@
 AR Path="/60D33366/61348F6E" Ref="#PWR?"  Part="1"
 AR Path="/61348F6E" Ref="#PWR?"  Part="1"
-AR Path="/6131300C/61348F6E" Ref="#PWR031"  Part="1"
-F 0 "#PWR031" H 6250 3800 50  0001 C CNN
+AR Path="/6131300C/61348F6E" Ref="#PWR0167"  Part="1"
+F 0 "#PWR0167" H 6250 3800 50  0001 C CNN
 F 1 "GND" H 6255 3877 50  0000 C CNN
 F 2 "" H 6250 4050 50  0001 C CNN
@@
 AR Path="/60D33366/61348F79" Ref="C?"  Part="1"
 AR Path="/61348F79" Ref="C?"  Part="1"
-AR Path="/6131300C/61348F79" Ref="C8"  Part="1"
-F 0 "C8" V 6500 3500 50  0000 L CNN
+AR Path="/6131300C/61348F79" Ref="C72"  Part="1"
+F 0 "C72" V 6500 3500 50  0000 L CNN
 F 1 "100n/16V/X7R" V 6400 3300 50  0000 L CNN
 F 2 "Capacitor_SMD:C_0402_1005Metric" H 6288 3400 50  0001 C CNN
@@
 AR Path="/60D33366/61348F83" Ref="#PWR?"  Part="1"
 AR Path="/61348F83" Ref="#PWR?"  Part="1"
-AR Path="/6131300C/61348F83" Ref="#PWR022"  Part="1"
-F 0 "#PWR022" H 5100 3800 50  0001 C CNN
+AR Path="/6131300C/61348F83" Ref="#PWR0161"  Part="1"
+F 0 "#PWR0161" H 5100 3800 50  0001 C CNN
 F 1 "GND" H 5105 3877 50  0000 C CNN
 F 2 "" H 5100 4050 50  0001 C CNN
@@
 P 5100 3400
 AR Path="/61348F8F" Ref="#PWR?"  Part="1"
-AR Path="/6131300C/61348F8F" Ref="#PWR021"  Part="1"
-F 0 "#PWR021" H 5100 3250 50  0001 C CNN
+AR Path="/6131300C/61348F8F" Ref="#PWR0160"  Part="1"
+F 0 "#PWR0160" H 5100 3250 50  0001 C CNN
 F 1 "+5V" H 5115 3573 50  0000 C CNN
 F 2 "" H 5100 3400 50  0001 C CNN
@@
 AR Path="/620639FD/61348F9C" Ref="#PWR?"  Part="1"
 AR Path="/61348F9C" Ref="#PWR?"  Part="1"
-AR Path="/6131300C/61348F9C" Ref="#PWR026"  Part="1"
-F 0 "#PWR026" H 6000 3250 50  0001 C CNN
+AR Path="/6131300C/61348F9C" Ref="#PWR0163"  Part="1"
+F 0 "#PWR0163" H 6000 3250 50  0001 C CNN
 F 1 "+3.3V" H 6015 3573 50  0000 C CNN
 F 2 "" H 6000 3400 50  0001 C CNN
@@
 AR Path="/620639FD/61348FA9" Ref="#PWR?"  Part="1"
 AR Path="/61348FA9" Ref="#PWR?"  Part="1"
-AR Path="/6131300C/61348FA9" Ref="#PWR030"  Part="1"
-F 0 "#PWR030" H 6250 3250 50  0001 C CNN
+AR Path="/6131300C/61348FA9" Ref="#PWR0166"  Part="1"
+F 0 "#PWR0166" H 6250 3250 50  0001 C CNN
 F 1 "+3.3V" H 6265 3573 50  0000 C CNN
 F 2 "" H 6250 3400 50  0001 C CNN
@@
 AR Path="/620639FD/6132182C" Ref="#PWR?"  Part="1"
 AR Path="/6132182C" Ref="#PWR?"  Part="1"
-AR Path="/6131300C/6132182C" Ref="#PWR019"  Part="1"
-F 0 "#PWR019" H 5100 2050 50  0001 C CNN
+AR Path="/6131300C/6132182C" Ref="#PWR0158"  Part="1"
+F 0 "#PWR0158" H 5100 2050 50  0001 C CNN
 F 1 "+3.3V" H 5115 2373 50  0000 C CNN
 F 2 "" H 5100 2200 50  0001 C CNN
@@
 P 6250 2200
 AR Path="/61321822" Ref="#PWR?"  Part="1"
-AR Path="/6131300C/61321822" Ref="#PWR028"  Part="1"
-F 0 "#PWR028" H 6250 2050 50  0001 C CNN
+AR Path="/6131300C/61321822" Ref="#PWR0164"  Part="1"
+F 0 "#PWR0164" H 6250 2050 50  0001 C CNN
 F 1 "+5V" H 6265 2373 50  0000 C CNN
 F 2 "" H 6250 2200 50  0001 C CNN
@@
 P 6000 2200
 AR Path="/6132181C" Ref="#PWR?"  Part="1"
-AR Path="/6131300C/6132181C" Ref="#PWR025"  Part="1"
-F 0 "#PWR025" H 6000 2050 50  0001 C CNN
+AR Path="/6131300C/6132181C" Ref="#PWR0162"  Part="1"
+F 0 "#PWR0162" H 6000 2050 50  0001 C CNN
 F 1 "+5V" H 6015 2373 50  0000 C CNN
 F 2 "" H 6000 2200 50  0001 C CNN
@@
 AR Path="/60D33366/61321814" Ref="#PWR?"  Part="1"
 AR Path="/61321814" Ref="#PWR?"  Part="1"
-AR Path="/6131300C/61321814" Ref="#PWR020"  Part="1"
-F 0 "#PWR020" H 5100 2600 50  0001 C CNN
+AR Path="/6131300C/61321814" Ref="#PWR0159"  Part="1"
+F 0 "#PWR0159" H 5100 2600 50  0001 C CNN
 F 1 "GND" H 5105 2677 50  0000 C CNN
 F 2 "" H 5100 2850 50  0001 C CNN
@@
 AR Path="/60D33366/6132180E" Ref="C?"  Part="1"
 AR Path="/6132180E" Ref="C?"  Part="1"
-AR Path="/6131300C/6132180E" Ref="C7"  Part="1"
-F 0 "C7" V 6500 2300 50  0000 L CNN
+AR Path="/6131300C/6132180E" Ref="C71"  Part="1"
+F 0 "C71" V 6500 2300 50  0000 L CNN
 F 1 "100n/16V/X7R" V 6400 2100 50  0000 L CNN
 F 2 "Capacitor_SMD:C_0402_1005Metric" H 6288 2200 50  0001 C CNN
@@
 AR Path="/60D33366/61321807" Ref="#PWR?"  Part="1"
 AR Path="/61321807" Ref="#PWR?"  Part="1"
-AR Path="/6131300C/61321807" Ref="#PWR029"  Part="1"
-F 0 "#PWR029" H 6250 2600 50  0001 C CNN
+AR Path="/6131300C/61321807" Ref="#PWR0165"  Part="1"
+F 0 "#PWR0165" H 6250 2600 50  0001 C CNN
 F 1 "GND" H 6255 2677 50  0000 C CNN
 F 2 "" H 6250 2850 50  0001 C CNN
@@
 P 5550 2550
 AR Path="/61321801" Ref="U?"  Part="1"
-AR Path="/6131300C/61321801" Ref="U3"  Part="1"
-F 0 "U3" H 5550 2875 50  0000 C CNN
+AR Path="/6131300C/61321801" Ref="U15"  Part="1"
+F 0 "U15" H 5550 2875 50  0000 C CNN
 F 1 "SN74LV1T126" H 5550 2784 50  0000 C CNN
 F 2 "Package_TO_SOT_SMD:SOT-23-5" H 5550 2300 50  0001 C CNN
