File: UIBoardStandalone.kicad_pcb (KiCad board)
At the start: 2 copper layers, 132 x 68.5 mm, 330 parts, among them J1 Conn_02x08_Odd_Even, J2 Conn_02x15_Odd_Even, SW1 Button_X, SW10 Button_6, SW11 Button_S, SW12 Button_7, SW13 Button_8, SW14 Button_9, SW15 Button_G, SW16 Button_Y, SW17 Button_0, SW18 Button_Z, SW2 Button_R, SW3 Button_1, SW4 Button_2, SW5 Button_3, SW6 Button_P, SW7 Button_M, SW8 Button_4, SW9 Button_5, U1 HD1077R, U10 HD1077R, U11 HD1077R, U12 HD1077R, U13 HD1077R, U14 HD1077R, U15 HD1077R, U16 HD1077R, U17 MM74C923WM, U2 HD1077R, U3 HD1077R, U4 HD1077R, U5 HD1077R, U6 HD1077R, U7 HD1077R, U8 HD1077R, U9 HD1077R

Commit message: - Wert und Footprint der LED Vorwiderstaende angepasst
Connections:
- net +5VA renamed Net-(J2-Pad30)
Changed lines of the file:
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@@
   (net 93 "Net-(D8-Pad2)")
   (net 94 "Net-(D9-Pad2)")
-  (net 95 +5VA)
+  (net 95 "Net-(J2-Pad30)")
   (net_class Default "Dies ist die voreingestellte Netzklasse."
     (clearance 0.1524)
@@
     (uvia_drill 0.1016)
     (add_net +5V)
-    (add_net +5VA)
     (add_net /ButtonA2GND)
     (add_net /Data_Encoder_Data_Available)
@@
     (add_net "Net-(J2-Pad27)")
     (add_net "Net-(J2-Pad29)")
+    (add_net "Net-(J2-Pad30)")
     (add_net "Net-(J2-Pad8)")
     (add_net "Net-(J2-Pad9)")
@@
       (net 94 "Net-(D9-Pad2)"))
     (pad 1 smd roundrect (at -0.7875 0 270) (size 0.875 0.95) (layers F.Cu F.Paste F.Mask) (roundrect_rratio 0.25)
-      (net 95 +5VA))
+      (net 95 "Net-(J2-Pad30)"))
     (model ${KISYS3DMOD}/Resistor_SMD.3dshapes/R_0603_1608Metric.wrl
       (at (xyz 0 0 0))
@@
       (net 93 "Net-(D8-Pad2)"))
     (pad 1 smd roundrect (at -0.7875 0 270) (size 0.875 0.95) (layers F.Cu F.Paste F.Mask) (roundrect_rratio 0.25)
-      (net 95 +5VA))
+      (net 95 "Net-(J2-Pad30)"))
     (model ${KISYS3DMOD}/Resistor_SMD.3dshapes/R_0603_1608Metric.wrl
       (at (xyz 0 0 0))
@@
       (net 92 "Net-(D7-Pad2)"))
     (pad 1 smd roundrect (at -0.7875 0 90) (size 0.875 0.95) (layers F.Cu F.Paste F.Mask) (roundrect_rratio 0.25)
-      (net 95 +5VA))
+      (net 95 "Net-(J2-Pad30)"))
     (model ${KISYS3DMOD}/Resistor_SMD.3dshapes/R_0603_1608Metric.wrl
       (at (xyz 0 0 0))
@@
       (net 91 "Net-(D6-Pad2)"))
     (pad 1 smd roundrect (at -0.7875 0 90) (size 0.875 0.95) (layers F.Cu F.Paste F.Mask) (roundrect_rratio 0.25)
-      (net 95 +5VA))
+      (net 95 "Net-(J2-Pad30)"))
     (model ${KISYS3DMOD}/Resistor_SMD.3dshapes/R_0603_1608Metric.wrl
       (at (xyz 0 0 0))
@@
       (net 90 "Net-(D5-Pad2)"))
     (pad 1 smd roundrect (at -0.7875 0 90) (size 0.875 0.95) (layers F.Cu F.Paste F.Mask) (roundrect_rratio 0.25)
-      (net 95 +5VA))
+      (net 95 "Net-(J2-Pad30)"))
     (model ${KISYS3DMOD}/Resistor_SMD.3dshapes/R_0603_1608Metric.wrl
       (at (xyz 0 0 0))
@@
     )
     (pad 30 thru_hole oval (at 2.54 -35.56 180) (size 1.7 1.7) (drill 1) (layers *.Cu *.Mask)
-      (net 95 +5VA))
+      (net 95 "Net-(J2-Pad30)"))
     (pad 29 thru_hole oval (at 0 -35.56 180) (size 1.7 1.7) (drill 1) (layers *.Cu *.Mask)
       (net 80 "Net-(J2-Pad29)"))
