File: BluetoothModule.sch (KiCad schematic (older format))
At the start: 13 parts, among them U17 BM83SM1-00TA

Commit message: Kleinigkeiten
Other:
- note added: "Wird das Modul als I2S Master betrieben, kann dessen MCLK Ausgang zur Frequenzversorgung \ndes Slaves verwendet werden. vgl. DS 6.5. Das Modul versorgt den MAX98089 mit Takt, \nso dass der Oszillator entfallen kann\n\nThe BM83 serves as a master to provide clock and frame synchronous signals for the master/slave data\nsynchronizations, as illustrated in the following figures. The MCLK is optional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"
- note removed: "Wird das Modul als I2S Master betrieben, kann dessen MCLK Ausgang zur Frequenzversorgung \ndes Slaves verwendet werden. Dies ist hier aber nicht der Fall, daher bleibt MCLK unbeschalten.\nvgl. DS 6.5. Vermutlich könnte das Modul den MAX98089 mit dem Takt versorgen, \nso dass der Oszillator für MAX98 entfallen kann\n\nThe BM83 serves as a master to provide clock and frame synchronous signals for t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"
Changed lines of the file:
@@
 For the I2C, I2S, and UART groups, each respective group's traces should run parallel\nwith as wide spacing as possible and be isolated from other groups with GND copper\nfoil. If isolation is not possible due to limited space, please at least increase the \ninterval between traces belonging to different groups.
 Text Notes 7000 6350 0    50   ~ 0
-Wird das Modul als I2S Master betrieben, kann dessen MCLK Ausgang zur Frequenzversorgung \ndes Slaves verwendet werden. Dies ist hier aber nicht der Fall, daher bleibt MCLK unbeschalten.\nvgl. DS 6.5. Vermutlich könnte das Modul den MAX98089 mit dem Takt versorgen, \nso dass der Oszillator für MAX98 entfallen kann\n\nThe BM83 serves as a master to provide clock and frame synchronous signals for the master/slave data\nsynchronizations, as illustrated in the following figures. The MCLK is optional and is not required if the\nexternal I2S device can drive its system clock on its own.\n\nMaster CLK is not part of the I2S standard, but is commonly included for synchronizing \nthe internal operation of the analog/digital converters.\nQuelle: https://en.wikipedia.org/wiki/I%C2%B2S
+Wird das Modul als I2S Master betrieben, kann dessen MCLK Ausgang zur Frequenzversorgung \ndes Slaves verwendet werden. vgl. DS 6.5. Das Modul versorgt den MAX98089 mit Takt, \nso dass der Oszillator entfallen kann\n\nThe BM83 serves as a master to provide clock and frame synchronous signals for the master/slave data\nsynchronizations, as illustrated in the following figures. The MCLK is optional and is not required if the\nexternal I2S device can drive its system clock on its own.\n\nMaster CLK is not part of the I2S standard, but is commonly included for synchronizing \nthe internal operation of the analog/digital converters.\nQuelle: https://en.wikipedia.org/wiki/I%C2%B2S
 $Comp
 L Device:R R46

Commit message: - Layout MAX98 - Audiostecker Belegung angepasst
Parts:
- added R49: 0R, Resistor_SMD:R_0402_1005Metric, symbol Device:R
- added SW1: SW_DIP_x01, Connector_PinHeader_2.54mm:PinHeader_1x02_P2.54mm_Vertical, symbol Switch:SW_DIP_x01
Connections:
- net GND: now also R49.1
- net at U17.31 (P3_4/UART_RTS): now also SW1.1
- new net: R49.2, SW1.2
- no-connect marks 33 -> 32
Other:
- note added: "GND -> TEST MODE\nGPIO P3_4 is used to enter Test mode during reset. If the user wants to use this pin to control external\nperipherals, care must be taken to ensure this pin is not pulled LOW and accidentally enters Test mode."
- note removed: "Hat P3_4 internen Pullup? GND -> TEST MODE\nGPIO P3_4 is used to enter Test mode during reset. If the user wants to use this pin to control external\nperipherals, care must be taken to ensure this pin is not pulled LOW and accidentally enters Test mode."
Changed lines of the file:
@@
 	2650 4400 2650 4750
 NoConn ~ 6400 3550
-NoConn ~ 6400 1850
-Text Notes -150 3150 0    50   ~ 0
-Hat P3_4 internen Pullup? GND -> TEST MODE\nGPIO P3_4 is used to enter Test mode during reset. If the user wants to use this pin to control external\nperipherals, care must be taken to ensure this pin is not pulled LOW and accidentally enters Test mode.
+Text Notes 10300 2250 0    50   ~ 0
+GND -> TEST MODE\nGPIO P3_4 is used to enter Test mode during reset. If the user wants to use this pin to control external\nperipherals, care must be taken to ensure this pin is not pulled LOW and accidentally enters Test mode.
 Wire Wire Line
 	3000 3750 3200 3750
@@
 Wire Wire Line
 	1950 1850 4400 1850
+$Comp
+L Device:R R49
+U 1 1 61D7F80E
+P 10300 2650
+F 0 "R49" H 10100 2600 50  0000 C CNN
+F 1 "0R" H 10050 2700 50  0000 C CNN
+F 2 "Resistor_SMD:R_0402_1005Metric" V 10340 2640 50  0001 C CNN
+F 3 "~" H 10300 2650 50  0001 C CNN
+	1    10300 2650
+	-1   0    0    1
+$EndComp
+$Comp
+L power:GND #PWR0185
+U 1 1 61D8065B
+P 10300 3000
+F 0 "#PWR0185" H 10300 2750 50  0001 C CNN
+F 1 "GND" H 10305 2827 50  0000 C CNN
+F 2 "" H 10300 3000 50  0001 C CNN
+F 3 "" H 10300 3000 50  0001 C CNN
+	1    10300 3000
+	1    0    0    -1
+$EndComp
+$Comp
+L Switch:SW_DIP_x01 SW1
+U 1 1 61D80D80
+P 9900 2400
+F 0 "SW1" H 9900 2667 50  0000 C CNN
+F 1 "SW_DIP_x01" H 9900 2576 50  0000 C CNN
+F 2 "Connector_PinHeader_2.54mm:PinHeader_1x02_P2.54mm_Vertical" H 9900 2400 50  0001 C CNN
+F 3 "~" H 9900 2400 50  0001 C CNN
+	1    9900 2400
+	1    0    0    -1
+$EndComp
+Wire Wire Line
+	6400 1850 9600 1850
+Wire Wire Line
+	9600 1850 9600 2400
+Wire Wire Line
+	10200 2400 10300 2400
+Wire Wire Line
+	10300 2400 10300 2500
+Wire Wire Line
+	10300 2800 10300 3000
 $EndSCHEMATC

Commit message: - Letzter Zwischenstand vor Branch. Alles außer Spannungsversorgung und Zündung ist vorerst fertig.
Parts:
- R49: footprint Resistor_SMD:R_0402_1005Metric -> Resistor_SMD:R_0603_1608Metric
- renumbered SW1 to J8
Other:
- note added: "GND -> TEST MODE\nGPIO P3_4 is used to enter Test mode during reset. \nIf the user wants to use this pin to control external\nperipherals, care must be taken to ensure this pin is \nnot pulled LOW and accidentally enters Test mode.\n\nAls unbestückte Stiftleiste 2,54 ausgeführt"
- note removed: "GND -> TEST MODE\nGPIO P3_4 is used to enter Test mode during reset. If the user wants to use this pin to control external\nperipherals, care must be taken to ensure this pin is not pulled LOW and accidentally enters Test mode."
- moved on the sheet: C73, C74, C75, C76, C77, D10, D9, J8, R45, R46, R47, R48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
