File: RTC.sch (KiCad schematic (older format))
At the start: 5 parts, among them U18 PCF85063A, Y1 9HT12

Commit message: - BT1 fixed
Parts:
- BT1: footprint Battery:BatteryHolder_MPD_BC2003_1x2032 -> TeKaDe:BAT-HLD-005-THM
Other:
- note added: "Änderungen:\n- RTC IC gewechselt jetzt mit Quarz\n- auf CR2032 gewechselt, THT auf BOTTOM"
- note removed: "Änderungen:\n- RTC IC gewechselt jetzt mit Quarz\n- auf CR2032 gewechselt, SMD auf BOTTOM"
Changed lines of the file:
@@
 F 0 "BT1" H 3908 4146 50  0000 L CNN
 F 1 "Battery" H 3908 4055 50  0000 L CNN
-F 2 "Battery:BatteryHolder_MPD_BC2003_1x2032" V 3800 4160 50  0001 C CNN
+F 2 "TeKaDe:BAT-HLD-005-THM" V 3800 4160 50  0001 C CNN
 F 3 "~" V 3800 4160 50  0001 C CNN
 	1    3800 4100
@@
 I2C_SDA
 Text Notes 4450 5800 0    50   ~ 0
-Änderungen:\n- RTC IC gewechselt jetzt mit Quarz\n- auf CR2032 gewechselt, SMD auf BOTTOM
+Änderungen:\n- RTC IC gewechselt jetzt mit Quarz\n- auf CR2032 gewechselt, THT auf BOTTOM
 Wire Wire Line
 	6650 4250 7600 4250

Commit message: - merged Lib updates
Parts:
- BT1: footprint TeKaDe:BAT-HLD-005-THM -> TeKaDe:BAT-HLD-003-SMT
Changed lines of the file:
@@
 F 0 "BT1" H 3908 4146 50  0000 L CNN
 F 1 "Battery" H 3908 4055 50  0000 L CNN
-F 2 "TeKaDe:BAT-HLD-005-THM" V 3800 4160 50  0001 C CNN
+F 2 "TeKaDe:BAT-HLD-003-SMT" V 3800 4160 50  0001 C CNN
 F 3 "~" V 3800 4160 50  0001 C CNN
 	1    3800 4100
