File: RaspberryPiCM4.sch (KiCad schematic (older format))
At the start: 20 parts, among them U6 CM4_Connectors_Part1, U7 CM4_Connectors_Part2

Commit message: checkpoint: new schema, old layout
Parts:
- removed U6: CM4_Connectors_Part1, TeKaDe:CM4-Part1, symbol CM4:CM4_Connectors_Part1
- removed U7: CM4_Connectors_Part2, TeKaDe:CM4-Part2, symbol CM4:CM4_Connectors_Part2
- added J7: USB_A, Connector_USB:USB_A_Molex_67643_Horizontal, symbol Connector:USB_A
- added U7: Compute_Module_4_Connectors, TeKaDe:Raspberry-Pi-4-Compute-Module, symbol CM4:Compute_Module_4_Connectors
Connections:
- wire segments 186 -> 200
Changed lines of the file:
@@
 $Descr A4 11693 8268
 encoding utf-8
-Sheet 4 9
+Sheet 4 8
 Title ""
 Date ""
@@
 	1    0    0    -1
 $EndComp
+$Comp
+L CM4:Compute_Module_4_Connectors U7
+U 1 1 622AF813
+P 2100 850
+F 0 "U7" H 3300 1137 60  0000 C CNN
+F 1 "Compute_Module_4_Connectors" H 3300 1031 60  0000 C CNN
+F 2 "TeKaDe:Raspberry-Pi-4-Compute-Module" H 2300 900 60  0001 L CNN
+F 3 "" H 2300 700 60  0001 L CNN
+	1    2100 850
+	1    0    0    -1
+$EndComp
+$Comp
+L CM4:Compute_Module_4_Connectors U7
+U 2 1 622B2EA9
+P 8900 850
+F 0 "U7" H 9900 1137 60  0000 C CNN
+F 1 "Compute_Module_4_Connectors" H 9900 1031 60  0000 C CNN
+F 2 "TeKaDe:Raspberry-Pi-4-Compute-Module" H 9100 900 60  0001 L CNN
+F 3 "" H 9100 700 60  0001 L CNN
+	2    8900 850
+	1    0    0    -1
+$EndComp
 Wire Wire Line
 	2100 850  2000 850
@@
 $EndComp
 $Comp
-L CM4:CM4_Connectors_Part1 U6
-U 1 1 629A08EC
-P 2100 850
-F 0 "U6" H 3300 1115 50  0000 C CNN
-F 1 "CM4_Connectors_Part1" H 3300 1024 50  0000 C CNN
-F 2 "TeKaDe:CM4-Part1" H 3050 1050 50  0001 C CNN
-F 3 "" H 3050 1050 50  0001 C CNN
-	1    2100 850
+L Connector:USB_A J7
+U 1 1 669C0DA2
+P 6550 950
+F 0 "J7" H 6607 1417 50  0000 C CNN
+F 1 "USB_A" H 6607 1326 50  0000 C CNN
+F 2 "Connector_USB:USB_A_Molex_67643_Horizontal" H 6700 900 50  0001 C CNN
+F 3 " ~" H 6700 900 50  0001 C CNN
+	1    6550 950
 	1    0    0    -1
 $EndComp
 $Comp
-L CM4:CM4_Connectors_Part2 U7
-U 1 1 629A6B87
-P 8900 850
-F 0 "U7" H 9900 1115 50  0000 C CNN
-F 1 "CM4_Connectors_Part2" H 9900 1024 50  0000 C CNN
-F 2 "TeKaDe:CM4-Part2" H 9500 1300 50  0001 C CNN
-F 3 "" H 9500 1300 50  0001 C CNN
-	1    8900 850
+L power:+5V #PWR0117
+U 1 1 669FB474
+P 7000 650
+F 0 "#PWR0117" H 7000 500 50  0001 C CNN
+F 1 "+5V" H 7015 823 50  0000 C CNN
+F 2 "" H 7000 650 50  0001 C CNN
+F 3 "" H 7000 650 50  0001 C CNN
+	1    7000 650
 	1    0    0    -1
 $EndComp
+Wire Wire Line
+	6850 750  7000 750
+Wire Wire Line
+	7000 750  7000 650
+Wire Wire Line
+	6850 950  7950 950
+Wire Wire Line
+	7950 950  7950 1050
+Wire Wire Line
+	7950 1050 8900 1050
+Wire Wire Line
+	6850 1050 7050 1050
+Wire Wire Line
+	7050 1050 7050 850
+Wire Wire Line
+	7050 850  8050 850
+Wire Wire Line
+	8050 850  8050 950
+Wire Wire Line
+	8050 950  8900 950
+Wire Wire Line
+	6550 1350 6550 1650
+Wire Wire Line
+	6550 1650 6500 1650
+Wire Wire Line
+	6450 1650 6450 1350
+$Comp
+L power:GND #PWR0168
+U 1 1 66A27290
+P 6500 1650
+F 0 "#PWR0168" H 6500 1400 50  0001 C CNN
+F 1 "GND" H 6505 1477 50  0000 C CNN
+F 2 "" H 6500 1650 50  0001 C CNN
+F 3 "" H 6500 1650 50  0001 C CNN
+	1    6500 1650
+	1    0    0    -1
+$EndComp
+Connection ~ 6500 1650
+Wire Wire Line
+	6500 1650 6450 1650
 $EndSCHEMATC

Commit message: layout first try
Connections:
- net I2C0_SCL: no longer R34.2, U7.80 (I2C_SCL0)
- net I2C0_SDA: no longer R32.2, U7.82 (I2C_SDA0)
- net GPIO9: no longer names the net of U7.40 (GPIO9)
- net UART3_RX: no longer names the net of U7.34 (GPIO5)
- net UART3_TX: no longer names the net of U7.54 (GPIO4)
- no-connect marks 112 -> 115
Changed lines of the file:
@@
 $Descr A4 11693 8268
 encoding utf-8
-Sheet 4 8
+Sheet 3 6
 Title ""
 Date ""
@@
 Wire Wire Line
 	1000 2050 2100 2050
-Text HLabel 6400 2750 2    50   Output ~ 0
-GPIO9
-Wire Wire Line
-	6400 2750 4500 2750
 Text HLabel 6400 2950 2    50   Input ~ 0
 GPIO10
@@
 Text HLabel 1000 5750 0    50   Input ~ 0
 RUN
-$Comp
-L Device:R R?
-U 1 1 60F86D30
-P 5600 4450
-AR Path="/64BEC8E8/60F86D30" Ref="R?"  Part="1"
-AR Path="/614D7E9D/60F86D30" Ref="R?"  Part="1"
-AR Path="/631EEDC8/60F86D30" Ref="R32"  Part="1"
-F 0 "R32" H 5670 4496 50  0000 L CNN
-F 1 "NA" H 5670 4405 50  0000 L CNN
-F 2 "Resistor_SMD:R_0402_1005Metric" V 5530 4450 50  0001 C CNN
-F 3 "~" H 5600 4450 50  0001 C CNN
-	1    5600 4450
-	-1   0    0    -1
-$EndComp
 Text Notes 700  7600 0    50   ~ 0
 Änderungen: \nAlle I2C Pullups hier, aber unbestückt (Pin 56/58/80/82 int. 1k8 PU)\nLogik von RUN input nun negiert!\nUART0 wurde zu UART3\nUART1 wurde zu UART0, da UART1 miniUART auf den gleichen Pins\n(vgl. https://www.raspberrypi.org/documentation/configuration/uart.md)\nUSB komplett entfernt, SSH zugriff via Wifi\nActivity LED hinzugefuegt\nPower LED nur als Testpoint\nGPIO9 entfernt, da BM83.MFB nicht benötigt\n\nFeststellungen: \n3,5A 5V Regler reicht leicht, auch inkl. 1,8 und 3,3V Ausgänge\nnEXTRST wird nicht verwendet\nQuelle CM4 Lib: https://github.com/Kedarius/RPi-CM4-Kicad
@@
 	6950 5600 6950 4200
 $Comp
-L Device:R R?
-U 1 1 60F94A2C
-P 5750 4450
-AR Path="/64BEC8E8/60F94A2C" Ref="R?"  Part="1"
-AR Path="/614D7E9D/60F94A2C" Ref="R?"  Part="1"
-AR Path="/631EEDC8/60F94A2C" Ref="R34"  Part="1"
-F 0 "R34" H 5820 4496 50  0000 L CNN
-F 1 "NA" H 5820 4405 50  0000 L CNN
-F 2 "Resistor_SMD:R_0402_1005Metric" V 5680 4450 50  0001 C CNN
-F 3 "~" H 5750 4450 50  0001 C CNN
-	1    5750 4450
-	1    0    0    -1
-$EndComp
-$Comp
 L CM4:Compute_Module_4_Connectors U7
 U 1 1 622AF813
@@
 	4700 4950 4500 4950
 Wire Wire Line
-	4500 4750 5750 4750
-Wire Wire Line
-	4500 4850 5600 4850
-Wire Wire Line
 	4500 3550 5750 3550
 Wire Wire Line
@@
 NoConn ~ 2100 3650
 Wire Wire Line
-	4500 3450 6400 3450
-Wire Wire Line
-	4500 2450 6400 2450
-Wire Wire Line
 	4600 2850 4600 3350
 Wire Wire Line
@@
 $EndComp
 $Comp
-L power:+3V3 #PWR069
-U 1 1 64274D33
-P 5600 4150
-F 0 "#PWR069" H 5600 4000 50  0001 C CNN
-F 1 "+3V3" V 5600 4350 50  0000 C CNN
-F 2 "" H 5600 4150 50  0001 C CNN
-F 3 "" H 5600 4150 50  0001 C CNN
-	1    5600 4150
-	1    0    0    -1
-$EndComp
-$Comp
-L power:+3V3 #PWR071
-U 1 1 64275A29
-P 5750 4150
-F 0 "#PWR071" H 5750 4000 50  0001 C CNN
-F 1 "+3V3" V 5750 4350 50  0000 C CNN
-F 2 "" H 5750 4150 50  0001 C CNN
-F 3 "" H 5750 4150 50  0001 C CNN
-	1    5750 4150
-	1    0    0    -1
-$EndComp
-Wire Wire Line
-	5600 4850 5600 4600
-Connection ~ 5600 4850
-Wire Wire Line
-	5600 4850 6400 4850
-Wire Wire Line
-	5750 4750 5750 4600
-Connection ~ 5750 4750
-Wire Wire Line
-	5750 4750 6400 4750
-Wire Wire Line
-	5600 4300 5600 4150
-Wire Wire Line
-	5750 4300 5750 4150
-$Comp
 L Device:R R?
 U 1 1 642990BB
@@
 NoConn ~ 10900 2850
 NoConn ~ 10900 2750
-NoConn ~ 8900 1050
-NoConn ~ 8900 950
 NoConn ~ 8900 850
 $Comp
@@
 Text HLabel 6400 3550 2    50   Output ~ 0
 I2C1_SCL
-Text HLabel 6400 2450 2    50   Input ~ 0
-UART3_RX
-Text HLabel 6400 3450 2    50   Output ~ 0
-UART3_TX
 Text HLabel 1000 3350 0    50   Input ~ 0
 UART0_RX
@@
 Wire Wire Line
 	6500 1650 6450 1650
+NoConn ~ 4500 2450
+NoConn ~ 4500 2750
+NoConn ~ 4500 3450
+NoConn ~ 4500 4750
+NoConn ~ 4500 4850
+Wire Wire Line
+	5750 4300 5750 4150
+Wire Wire Line
+	5600 4300 5600 4150
+$Comp
+L power:+3V3 #PWR071
+U 1 1 64275A29
+P 5750 4150
+F 0 "#PWR071" H 5750 4000 50  0001 C CNN
+F 1 "+3V3" V 5750 4350 50  0000 C CNN
+F 2 "" H 5750 4150 50  0001 C CNN
+F 3 "" H 5750 4150 50  0001 C CNN
+	1    5750 4150
+	1    0    0    -1
+$EndComp
+$Comp
+L power:+3V3 #PWR069
+U 1 1 64274D33
+P 5600 4150
+F 0 "#PWR069" H 5600 4000 50  0001 C CNN
+F 1 "+3V3" V 5600 4350 50  0000 C CNN
+F 2 "" H 5600 4150 50  0001 C CNN
+F 3 "" H 5600 4150 50  0001 C CNN
+	1    5600 4150
+	1    0    0    -1
+$EndComp
+$Comp
+L Device:R R?
+U 1 1 60F94A2C
+P 5750 4450
+AR Path="/64BEC8E8/60F94A2C" Ref="R?"  Part="1"
+AR Path="/614D7E9D/60F94A2C" Ref="R?"  Part="1"
+AR Path="/631EEDC8/60F94A2C" Ref="R34"  Part="1"
+F 0 "R34" H 5820 4496 50  0000 L CNN
+F 1 "NA" H 5820 4405 50  0000 L CNN
+F 2 "Resistor_SMD:R_0402_1005Metric" V 5680 4450 50  0001 C CNN
+F 3 "~" H 5750 4450 50  0001 C CNN
+	1    5750 4450
+	1    0    0    -1
+$EndComp
+$Comp
+L Device:R R?
+U 1 1 60F86D30
+P 5600 4450
+AR Path="/64BEC8E8/60F86D30" Ref="R?"  Part="1"
+AR Path="/614D7E9D/60F86D30" Ref="R?"  Part="1"
+AR Path="/631EEDC8/60F86D30" Ref="R32"  Part="1"
+F 0 "R32" H 5670 4496 50  0000 L CNN
+F 1 "NA" H 5670 4405 50  0000 L CNN
+F 2 "Resistor_SMD:R_0402_1005Metric" V 5530 4450 50  0001 C CNN
+F 3 "~" H 5600 4450 50  0001 C CNN
+	1    5600 4450
+	-1   0    0    -1
+$EndComp
 $EndSCHEMATC
